File: hardware/modulmag/modulmag.kicad_sch (KiCad schematic)
At the start: 52 parts, among them J1 DEBUG, J2 BUS_IN, J3 BUS_OUT, J4 BŐVÍTŐ, U1 P78E05-1000, U2 ISO1042BDWV, U3 ESD2CAN24-Q1, U5 NCP1117ST33T3G, U6 STM32F303RET6, Y1 8MHz

Commit message: Hardver: központi 5 V, közös föld, 12–26 V, HW-ID 16 sáv (D71)
Vezérlő: LMR33630 (5,2 V) + LM66200 (USB-vel VAGY-olva) + TPS259531 eFuse (2 A);
F1 2 A, D1 B360 a 12 V-os működéshez. Modulmag: táp a buszról (AP2112K), TCAN1044AV,
nincs izoláció, PC1 = VBUS_SENSE. LED/relé: VIN_SENSE a PB11-en, relémodul saját
tekercs-táppal. Bemeneti modul: nincs 24 V. HW-ID/HW_REV 16 sáv. Specifikációk,
áttekintés, beszerzés, ütemterv frissítve.

Co-Authored-By: Claude Opus 5.5 <noreply@anthropic.com>
Parts:
- removed C1: 10µ/50V, Capacitor_SMD:C_1210_3225Metric, symbol Device:C
- removed C12: 47µ/50V, Capacitor_SMD:CP_Elec_6.3x7.7, symbol Device:C_Polarized
- removed C3: 10µ tantál, Capacitor_Tantalum_SMD:CP_EIA-3216-18_Kemet-A, symbol Device:C_Polarized
- removed D1: SS16, Diode_SMD:D_SMA, symbol Device:D_Schottky
- removed D2: SMBJ28A, Diode_SMD:D_SMB, symbol Device:D_Zener
- removed D6: SS14, Diode_SMD:D_SMA, symbol Device:D_Schottky
- removed F1: 0,5A, Fuse:Fuse_1206_3216Metric, symbol Device:Fuse
- removed JP2: GND_BUS–GND, Jumper:SolderJumper-2_P1.3mm_Open_RoundedPad1.0x1.5mm, symbol Jumper:SolderJumper_2_Open
- removed R6: 0R, Resistor_SMD:R_1206_3216Metric, symbol Device:R
- removed U1: P78E05-1000, Converter_DCDC:Converter_DCDC_RECOM_R-78E-0.5_THT, symbol Converter_DCDC:R-78E5.0-1.0
- removed U2: ISO1042BDWV, Package_SO:SOIC-8_7.5x5.85mm_P1.27mm, symbol modularis:ISO1042BDWV
- removed U5: NCP1117ST33T3G, Package_TO_SOT_SMD:SOT-223-3_TabPin2, symbol Regulator_Linear:NCP1117-3.3_SOT223
- added C3: 10µ, Capacitor_SMD:C_0805_2012Metric, symbol Device:C
- added R12: 0R, Resistor_SMD:R_0603_1608Metric, symbol Device:R
- added U2: TCAN1044AVDRQ1, Package_SO:SOIC-8_3.9x4.9mm_P1.27mm, symbol Interface_CAN_LIN:MCP2562-E-SN
- added U5: AP2112K-3.3TRG1, Package_TO_SOT_SMD:SOT-23-5, symbol Regulator_Linear:AP2112K-3.3
- C2: value 22µ/10V -> 10µ; footprint Capacitor_SMD:C_1206_3216Metric -> Capacitor_SMD:C_0805_2012Metric; Megjegyzés (none) -> X7R, 16 V – a buszról érkező 5 V puffere
- R10: Megjegyzés revízió: v1-en üres (0. sáv); később a HW-ID sávjai szerint -> felső ellenállás mindig 10 k; az alsó adja a revíziót (16 s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; now fitted
- R11: value 10k 1% -> 715R 1%; Megjegyzés (none) -> v1 = 1. sáv (0,22 V); csak R10: 15. sáv = a firmware-ből me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
- R3: value 150k -> 10k 1%
- R4: value 10k -> 10k 1%
Connections:
- net +24V_P is gone; now on net +5V: R3.1
- net GND_BUS is gone; now on net GND: C18.2, C19.2, D5.2 (A), J2.2 (Pin_2), J3.2 (Pin_2), U3.3 (A)
- net V_BUS_P is gone; now on net +5V: C18.1, C19.1, D5.1 (K), J2.1 (Pin_1), J3.1 (Pin_1)
- net +3V3: now also C3.1, U2.5 (Vio), U5.5 (VOUT)
- net +5V: now also U2.3 (VDD), U5.1 (VIN), U5.3 (EN)
- net CAN_H: now also U2.7 (CANH)
- net CAN_L: now also U2.6 (CANL)
- net CAN_RX: now also U2.4 (RXD)
- net CAN_TX: now also U2.1 (TXD)
- net GND: now also C3.2, R12.2, U2.2 (VSS), U5.2 (GND)
- net VIN_SENSE renamed VBUS_SENSE
- new net: R12.1, U2.8 (STBY)
- no-connect marks 9 -> 10
Other:
- note added: "+5V TVS · CAN ESD · lezárás (JP1: csak a lánc két végén)"
- note added: "1. TÁP: a busz +5V-ja (J2/J3, 1-es tű) → U5 AP2112K-3.3 (kis ejtésű LDO) → +3V3"
- note added: "3. CAN – U2 TCAN1044AVDRQ1 (MCP2562 szimbólum, lábról lábra azonos): VCC = +5V (busz), VIO = +3V3"
- note added: "4. BUSZ: J2 és J3 azonos tűi átmenők (1 +5V · 2 GND · 3 CAN_L · 4 CAN_H); ESD és TVS a csatlakozók mellé"
- note added: "BŐVÍTÉS (D69, D71) – HW_REV: NYÁK-revízió a PB0-n (v1: 10k / 715 Ω → 1. sáv) · J4: DNP bővítő-tüskesor"
- note added: "D71: központi 5 V a vezérlőről, közös föld; 24 V a modulmagon nincs (a LED- és a relélap maga méri)"
- note added: "D71: közös föld – izoláció nincs; a vezérlő és minden modul egy tápról, csillagpontosan"
- note added: "VBUS_SENSE: 5 V → 2,5 V (PC1)"
- note removed: "1. TÁP: +24V_IN → F1 → D1 → R6 → +24V_P → U1 P78E05 (5 V) → U5 NCP1117 (3,3 V)"
- note removed: "3. IZOLÁLT CAN – ISO1042BDWV: a tok alatt minden rétegen rézmentes rés"
- note removed: "4. BUSZ-OLDAL (GND_BUS): J2 és J3 azonos tűi átmenők; ESD és TVS a csatlakozók mellé"
- note removed: "BUSZOS TÁP (D66, opció): D6 + JP2 beforrasztva → 24 V nélkül"
- note removed: "BŐVÍTÉS (D69) – HW_REV: NYÁK-revízió a PB0-n (v1: csak R11 → 0. sáv) · J4: DNP bővítő-tüskesor"
- note removed: "D56, D57 – a C12 elkó kötelező; a 24 V-os tápot ≤ 26 V-ra! (a P78E05 max. 36 V)"
- note removed: "VIN_SENSE: 24 V → 1,5 V (PC1)"
- note removed: "V_BUS TVS · CAN ESD · lezárás (JP1: csak a lánc két végén)"
- note removed: "a V_BUS-ról jár (izoláció nélkül!)"
- note removed: "logikai oldal (GND) busz-oldal (GND_BUS)"
- title: Modulmag – STM32F303RET6, izolált CAN, 24 → 5 → 3,3 V -> Modulmag – STM32F303RET6, CAN, táp a buszról (+5V → 3,3 V)
