File: hardware/vezerlo/vezerlo.kicad_sch (KiCad schematic)
At the start: 0 parts

Commit message: Hardver: modulmag + vezérlő kapcsolási rajz (vázlat, ERC tiszta)
Elektromosan a MODULMAG-SPEC és a VEZERLO-SPEC szerint, elrendezés nélkül.
Közös könyvtár: saját szimbólumok, ESP32-C6-WROOM-1/-1U footprint (Espressif,
CC-BY-SA, licenc a lib/-ben). A KiCad .history/ mappája gitignore-ba.

Co-Authored-By: Claude Opus 5.5 <noreply@anthropic.com>
Parts:
- added C1: 47µ/50V, Capacitor_SMD:CP_Elec_6.3x7.7, symbol Device:C_Polarized
- added C10, C11, C12, C13: 22µ/10V, Capacitor_SMD:C_1206_3216Metric, symbol Device:C
- added C14, C23, C24, C27, C3, C31, C32, C33, C34, C35, C36, C37, C42, C44, C45, C46, C7: 100n, Capacitor_SMD:C_0603_1608Metric, symbol Device:C
- added C15, C21, C22, C43: 1µ, Capacitor_SMD:C_0603_1608Metric, symbol Device:C
- added C16, C30: 10n, Capacitor_SMD:C_0603_1608Metric, symbol Device:C
- added C17, C19: 6,8n, Capacitor_SMD:C_0603_1608Metric, symbol Device:C
- added C18: 22n, Capacitor_SMD:C_0603_1608Metric, symbol Device:C
- added C2: 10µ/50V, Capacitor_SMD:C_1210_3225Metric, symbol Device:C
- added C20: 1n/2kV, Capacitor_SMD:C_1206_3216Metric, symbol Device:C
- added C25: 10µ/16V, Capacitor_SMD:C_0805_2012Metric, symbol Device:C
- added C26: 22µ, Capacitor_SMD:C_0805_2012Metric, symbol Device:C
- added C28: DNP, Capacitor_SMD:C_0603_1608Metric, symbol Device:C
- added C29: 4µ7, Capacitor_SMD:C_0805_2012Metric, symbol Device:C
- added C38, C39: 10µ, Capacitor_SMD:C_0805_2012Metric, symbol Device:C
- added C4: 4µ7/50V, Capacitor_SMD:C_1210_3225Metric, symbol Device:C
- added C40, C41: 18p, Capacitor_SMD:C_0603_1608Metric, symbol Device:C
- added C5, C6: 220n/50V, Capacitor_SMD:C_0603_1608Metric, symbol Device:C
- added C8: 1µ/16V, Capacitor_SMD:C_0603_1608Metric, symbol Device:C
- added C9: 20p, Capacitor_SMD:C_0603_1608Metric, symbol Device:C
- added D1, D8: SS16, Diode_SMD:D_SMA, symbol Device:D_Schottky
- added D2, D7: SMBJ28A, Diode_SMD:D_SMB, symbol Device:D_Zener
- added D3: B360, Diode_SMD:D_SMC, symbol Device:D_Schottky
- added D4: SMF5.0A, Diode_SMD:D_SOD-123F, symbol Device:D_Zener
- added D5: zöld, LED_SMD:LED_0603_1608Metric, symbol Device:LED
- added D6: WS2812B-V5, LED_SMD:LED_WS2812B_PLCC4_5.0x5.0mm_P3.2mm, symbol LED:WS2812B
- added D9: BAT54WS, Diode_SMD:D_SOD-323, symbol Device:D_Schottky
- added F1: 1A, Fuse:Fuse_1206_3216Metric, symbol Device:Fuse
- added FB1: 120R@100MHz, Inductor_SMD:L_0603_1608Metric, symbol Device:FerriteBead_Small
- added J1: 24V IN, TerminalBlock_Phoenix:TerminalBlock_Phoenix_PT-1,5-2-3.5-H_1x02_P3.50mm_Horizontal, symbol Connector_Generic:Conn_01x02
- added J2, J3: BUS (XH), Connector_JST:JST_XH_B4B-XH-A_1x04_P2.50mm_Vertical, symbol Connector_Generic:Conn_01x04
- added J4: USB-C 16P, Connector_USB:USB_C_Receptacle_HRO_TYPE-C-31-M-12, symbol Connector:USB_C_Receptacle_USB2.0_16P
- added J5: DEBUG, Connector_PinHeader_2.54mm:PinHeader_1x06_P2.54mm_Vertical, symbol Connector_Generic:Conn_01x06
- added J6: HR911105A, Connector_RJ:RJ45_Hanrun_HR911105A_Horizontal, symbol Connector:RJ45_Hanrun_HR911105A_Horizontal
- added JP1: LEZÁRÁS, Connector_PinHeader_2.54mm:PinHeader_1x02_P2.54mm_Vertical, symbol Jumper:Jumper_2_Open
- added JP2: VCC: 1-2=5V / 2-3=3V3, Jumper:SolderJumper-3_P1.3mm_Bridged12_RoundedPad1.0x1.5mm, symbol Jumper:SolderJumper_3_Bridged12
- added JP3: VIO: 1-2=3V3 / 2-3=GND, Jumper:SolderJumper-3_P1.3mm_Bridged12_RoundedPad1.0x1.5mm, symbol Jumper:SolderJumper_3_Bridged12
- added L1: 6,8µH, Inductor_SMD:L_Coilcraft_XAL5030-XXX, symbol Device:L
- added R1: 150k, Resistor_SMD:R_0603_1608Metric, symbol Device:R
- added R10: 470k, Resistor_SMD:R_0603_1608Metric, symbol Device:R
- added R11: 47k, Resistor_SMD:R_0603_1608Metric, symbol Device:R
- added R12: 61,9k 1%, Resistor_SMD:R_0603_1608Metric, symbol Device:R
- added R13: 100k, Resistor_SMD:R_0603_1608Metric, symbol Device:R
- added R14: 22k, Resistor_SMD:R_0603_1608Metric, symbol Device:R
- added R15, R16, R17, R18, R2, R34, R35, R36, R37, R38: 10k, Resistor_SMD:R_0603_1608Metric, symbol Device:R
- added R19, R32, R33, R43: 0R, Resistor_SMD:R_0603_1608Metric, symbol Device:R
- added R20, R21, R22, R23: 49,9R 1%, Resistor_SMD:R_0603_1608Metric, symbol Device:R
- added R24: 10R 1%, Resistor_SMD:R_0603_1608Metric, symbol Device:R
- added R25: 120R, Resistor_SMD:R_0805_2012Metric, symbol Device:R
- added R26, R27: 22R, Resistor_SMD:R_0603_1608Metric, symbol Device:R
- added R28, R29: 5,1k, Resistor_SMD:R_0603_1608Metric, symbol Device:R
- added R3: 100k 1%, Resistor_SMD:R_0603_1608Metric, symbol Device:R
- added R30, R44: 2,2k, Resistor_SMD:R_0603_1608Metric, symbol Device:R
- added R31: 33R, Resistor_SMD:R_0603_1608Metric, symbol Device:R
- added R39: 499R, Resistor_SMD:R_0603_1608Metric, symbol Device:R
- added R4: 43,2k 1%, Resistor_SMD:R_0603_1608Metric, symbol Device:R
- added R40: 12,4k 1%, Resistor_SMD:R_0603_1608Metric, symbol Device:R
- added R41, R42: 330R, Resistor_SMD:R_0603_1608Metric, symbol Device:R
- added R7: 10R, Resistor_SMD:R_2512_6332Metric, symbol Device:R
- added SW1: RESET, Button_Switch_SMD:SW_SPST_TL3342, symbol Switch:SW_Push
- added SW2: BOOT, Button_Switch_SMD:SW_SPST_TL3342, symbol Switch:SW_Push
- added TP1: GPIO4, TestPoint:TestPoint_Pad_D1.5mm, symbol Connector:TestPoint
- added TP2: GPIO5, TestPoint:TestPoint_Pad_D1.5mm, symbol Connector:TestPoint
- added TP3: GPIO22, TestPoint:TestPoint_Pad_D1.5mm, symbol Connector:TestPoint
- added TP4: GPIO23, TestPoint:TestPoint_Pad_D1.5mm, symbol Connector:TestPoint
- added U1: LMR36015BRNXR, symbol modularis:LMR36015BRNXR
- added U2: P78E05-1000, Converter_DCDC:Converter_DCDC_RECOM_R-78E-0.5_THT, symbol Converter_DCDC:R-78E5.0-1.0
- added U3: TPS2553DBVR, Package_TO_SOT_SMD:SOT-23-6, symbol modularis:TPS2553DBV
- added U4: ESP32-C6-WROOM-1-N16, modularis:ESP32-C6-WROOM-1, symbol modularis:ESP32-C6-WROOM-1
- added U5: W5500, Package_QFP:LQFP-48_7x7mm_P0.5mm, symbol Interface_Ethernet:W5500
- added U6: TCAN1044AVDRQ1, Package_SO:SOIC-8_3.9x4.9mm_P1.27mm, symbol Interface_CAN_LIN:MCP2562-E-SN
- added U7: ESD2CAN24-Q1, Package_TO_SOT_SMD:SOT-23, symbol Power_Protection:NUP2105L
- added U8: USBLC6-2SC6, Package_TO_SOT_SMD:SOT-23-6, symbol Power_Protection:USBLC6-2SC6
- added U9: 74HCT14D, Package_SO:SOIC-14_3.9x8.7mm_P1.27mm, symbol 74xx:74HC14
- added Y1: 25MHz ±30ppm, Crystal:Crystal_SMD_3225-4Pin_3.2x2.5mm, symbol Device:Crystal_GND24
Connections:
- new net +24V_F: C1.1, C2.1, D7.1 (K), R7.2, U2.1 (IN)
- new net +24V_F1: D1.2 (A), F1.2
- new net +24V_IN: F1.1, J1.1 (Pin_1)
- new net +24V_P: D1.1 (K), D2.1 (K), D8.2 (A), R1.1, R10.1, R7.1
- new net +3V3: C10.1, C11.1, C12.1, C26.1, C27.1, C37.1, C38.1, C9.1, FB1.1, JP2.3 (B), JP3.1 (A), L1.2, R15.1, R16.1, R17.1, R18.1, R3.1, R33.1, R34.1, R35.1, R36.1, R37.1, R38.1, R41.1, R42.1, R44.1, U4.2 (3V3), U5.28 (VDD)
- new net +3V3A: C16.1, C31.1, C32.1, C33.1, C34.1, C35.1, C36.1, C39.1, FB1.2, R20.2, R21.2, R24.1, U5.11 (AVDD), U5.15 (AVDD), U5.17 (AVDD), U5.21 (AVDD), U5.4 (AVDD), U5.8 (AVDD)
- new net +5V: C13.1, C22.1, C23.1, C45.1, C46.1, D6.1 (VDD), JP2.1 (A), U2.3 (OUT), U3.1 (IN), U9.14 (VCC)
- new net BOOT: J5.6 (Pin_6), R16.2, SW2.1, U4.15 (GPIO9)
- new net BUCK_BOOT: C7.1, U1.4 (BOOT)
- new net BUCK_FB: C9.2, R3.2, R4.1, U1.7 (FB)
- new net BUCK_SW: C7.2, L1.1, U1.12 (SW), U1.3 (NC)
- new net BUCK_VCC: C8.1, U1.5 (VCC)
- new net CAN_H: J2.4 (Pin_4), J3.4 (Pin_4), JP1.1 (A), U6.7 (CANH), U7.2 (K)
- new net CAN_L: J2.3 (Pin_3), J3.3 (Pin_3), R25.2, U6.6 (CANL), U7.1 (K)
- new net CAN_RX: U4.17 (GPIO19), U6.4 (RXD)
- new net CAN_STB: R43.1, U6.8 (STBY)
- new net CAN_TERM: JP1.2 (B), R25.1
- new net CAN_TX: R35.2, U4.16 (GPIO18), U6.1 (TXD)
- new net CAN_VCC: C42.1, C43.1, JP2.2 (C), U6.3 (VDD)
- new net CAN_VIO: C44.1, JP3.2 (C), U6.5 (Vio)
- new net CHIP_EN: C15.1, J5.5 (Pin_5), R15.2, SW1.1, U4.3 (EN/CHIP_PU)
- new net ETH_LED_ACT: J6.11, U5.27 (ACTLED)
- new net ETH_LED_G_A: J6.9, R41.2
- new net ETH_LED_LINK: J6.10, U5.25 (LINKLED)
- new net ETH_LED_Y_A: J6.12, R42.2
- new net ETH_RCT: C19.1, J6.5 (RCT)
- new net ETH_RXB: C17.1, R22.2, R23.2
- new net ETH_RXN: J6.6 (RD-), R23.1, U5.5 (RXN)
- new net ETH_RXP: J6.3 (RD+), R22.1, U5.6 (RXP)
- new net ETH_SHIELD: C20.1, J6.SH
- new net ETH_TCT: C18.1, J6.4 (TCT), R24.2
- new net ETH_TXN: J6.2 (TD-), R21.1, U5.1 (TXN)
- new net ETH_TXP: J6.1 (TD+), R20.1, U5.2 (TXP)
- new net GND: C1.2, C10.2, C11.2, C12.2, C13.2, C14.2, C15.2, C16.2, C17.2, C18.2, C19.2, C2.2, C20.2, C21.2, C22.2, C23.2, C24.2, C25.2, C26.2, C27.2, C28.2, C29.2, C3.2, C30.2, C31.2, C32.2, C33.2, C34.2, C35.2, C36.2, C37.2, C38.2, C39.2, C4.2, C40.2, C41.2, C42.2, C43.2, C44.2, C45.2, C46.2, C5.2, C6.2, C8.2, D2.2 (A), D4.2 (A), D5.1 (K), D6.3 (VSS), D7.2 (A), J1.2 (Pin_2), J2.2 (Pin_2), J3.2 (Pin_2), J4.A1 (GND), J4.A12 (GND), J4.B1 (GND), J4.B12 (GND), J4.SH (SHIELD), J5.2 (Pin_2), J6.8, JP3.3 (B), R11.2, R12.2, R14.2, R2.2, R28.2, R29.2, R30.2, R4.2, R40.2, R43.2, SW1.2, SW2.2, U1.1 (PGND), U1.11 (PGND), U1.6 (AGND), U1.8 (PG), U2.2 (GND), U3.2 (GND), U4.1 (GND), U4.28 (GND), U4.29 (GND), U5.14 (AGND), U5.16 (AGND), U5.19 (AGND), U5.23 (RSVD), U5.29 (GND), U5.3 (AGND), U5.48 (AGND), U5.9 (AGND), U6.2 (VSS), U7.3 (A), U8.2 (GND), U9.11, U9.13, U9.5, U9.7 (GND), U9.9, Y1.2 (G), Y1.4 (G)
- new net GPIO15: R18.2, U4.23 (GPIO15)
- new net GPIO22: TP3.1, U4.20 (GPIO22)
- new net GPIO23: TP4.1, U4.21 (GPIO23)
- new net GPIO4: TP1.1, U4.4 (MTMS/GPIO4/ADC1_CH4)
- new net GPIO5: TP2.1, U4.5 (MTDI/GPIO5/ADC1_CH5)
- new net J5_VREF: J5.1 (Pin_1), R33.2
- new net LED_PWR: D5.2 (A), R44.2
- new net RGB_DIN: D6.4 (DIN), R31.2, R32.2
- new net RGB_DIN_3V3: R17.2, R32.1, U4.10 (GPIO8), U9.1
- new net RGB_DIN_5V: R31.1, U9.4
- new net RGB_HCT_MID: U9.2, U9.3
- new net SPI_MISO: U4.27 (GPIO2/ADC1_CH2), U5.34 (MISO)
- new net SPI_MOSI: U4.7 (MTDO/GPIO7), U5.35 (MOSI)
- new net SPI_SCLK: C28.1, R19.2, U5.33 (SCLK)
- new net SPI_SCLK_C6: R19.1, U4.6 (MTCK/GPIO6/ADC1_CH6)
- new net U0RXD: J5.4 (Pin_4), U4.24 (U0RXD/GPIO17)
- new net U0TXD: J5.3 (Pin_3), R39.2
- new net U0TXD_C6: R39.1, U4.25 (U0TXD/GPIO16)
- new net USB_CC1: J4.A5 (CC1), R28.1
- new net USB_CC2: J4.B5 (CC2), R29.1
- new net USB_DM: R27.2, U4.13 (GPIO12/USB_D-)
- new net USB_DM_CONN: J4.A7 (D-), J4.B7 (D-), R27.1, U8.3 (I/O2), U8.4 (I/O2)
- new net USB_DP: R26.2, U4.14 (GPIO13/USB_D+)
- new net USB_DP_CONN: J4.A6 (D+), J4.B6 (D+), R26.1, U8.1 (I/O1), U8.6 (I/O1)
- new net VBUS_EN: D9.1 (K), U4.18 (GPIO20)
- new net VBUS_EN_IN: D9.2 (A), R10.2, R11.1, U3.3 (EN)
- new net VBUS_FAULT: R34.2, U3.4 (~{FAULT}), U4.19 (GPIO21)
- new net VBUS_ILIM: R12.1, U3.5 (ILIM)
- new net VBUS_SENSE: C14.1, R13.2, R14.1, U4.9 (GPIO1/ADC1_CH1/XTAL_32K_N)
- new net VIN_BUCK: C4.1, C5.1, C6.1, D3.1 (K), D8.1 (K), U1.10 (VIN), U1.2 (VIN), U1.9 (EN)
- new net VIN_SENSE: C3.1, R1.2, R2.1, U4.8 (GPIO0/ADC1_CH0/XTAL_32K_P)
- new net VUSB: C21.1, D3.2 (A), J4.A4 (VBUS), J4.A9 (VBUS), J4.B4 (VBUS), J4.B9 (VBUS), R30.1, U8.5 (VBUS)
- new net V_BUS: C24.1, C25.1, D4.1 (K), J2.1 (Pin_1), J3.1 (Pin_1), R13.1, U3.6 (OUT)
- new net W5500_CS: R36.2, U4.11 (GPIO10), U5.32 (~{SCS})
- new net W5500_INT: R38.2, U4.26 (GPIO3/ADC1_CH3), U5.36 (~{INT})
- new net W5500_RST: R37.2, U4.12 (GPIO11), U5.37 (~{RST})
- new net W_1V2O: C30.1, U5.22 (1V2O)
- new net W_EXRES: R40.1, U5.10 (EXRES1)
- new net W_TOCAP: C29.1, U5.20 (TOCAP)
- new net XTAL25_I: C40.1, U5.30 (XI/CLKIN), Y1.1
- new net XTAL25_O: C41.1, U5.31 (XO), Y1.3
- no-connect marks 0 -> 25
Other:
- note added: "2.1 BEMENET: +24V_IN → F1 → D1 → +24V_P; USB csak a 3,3 V-os buckot táplálja (D3) – a V_BUS USB-ről hardveresen KI (D61)"
- note added: "2.2 3,3 V – LMR36015BRNXR (1 MHz): FOOTPRINT a TI Ultra Librarian-ből!"
- note added: "2.4 V_BUS – TPS2553: EN osztó a +24V_P-ről (csak 24 V mellett BE), GPIO20 BAT54-en át letiltja"
- note added: "3. ESP32-C6-WROOM-1-N16 (fém szekrénybe -1U – az EPAD helyét ellenőrizni!)"
- note added: "4. ETHERNET – W5500 + HR911105A MagJack (opcionálisan beültetve; MDI a WIZnet use_mag referencia szerint)"
- note added: "5–6. CAN – TCAN1044AVDRQ1 (MCP2562 szimbólum, lábról lábra azonos) · JP2 alap 5V: 1044/2562 · 3V3: 330/230"
- note added: "7. USB-C – csak eszköz, csak táp-fogyasztó (CC1/CC2 külön 5,1 kΩ)"
- note added: "8. GOMBOK, LED-EK, DEBUG – U9 és R32 egyszerre NE legyen beültetve"
- note added: "VBG (18) NYITVA · RSVD 38–42 NYITVA · RSVD 23 GND · PMODE nyitva (auto-negotiation)"
- note added: "VÁZLAT – generálva a VEZERLO-SPEC.md alapján (2026-10-14). Elrendezést rendezd; a bekötés címkékkel kész."
- title: Vezérlő (ESP32-C6) -> Vezérlő – ESP32-C6-WROOM-1 + W5500 + CAN + V_BUS

Commit message: Hardver: mind az öt kapcsolási rajz elrendezve (vezetékes, blokkos), netlista-ellenőrzővel
Funkcionális blokkok, balról jobbra jelút, tápsín felül / GND alul; blokkon belül
vezeték, blokkok között és az IC-lábakon címke. kigen: lábpozíció, place(),
wire/junction/rail, tükrözés, 1,27 mm-es rács, olvasható mezők. gen/netcmp.py:
két netlista lábszintű összevetése – a bekötés az átrendezés előttivel azonos
(a modulmag D66-os D6/JP2-jét kivéve). ERC: 0 hiba mind az öt lapon.

Co-Authored-By: Claude Opus 5.5 <noreply@anthropic.com>
Parts:
- D5: Megjegyzés (none) -> táp-LED
Connections:
- net +24V_F1: no longer names the net of D1.2 (A), F1.2
- net BUCK_BOOT: no longer names the net of C7.1, U1.4 (BOOT)
- net BUCK_FB: no longer names the net of C9.2, R3.2, R4.1, U1.7 (FB)
- net BUCK_SW: no longer names the net of C7.2, L1.1, U1.12 (SW), U1.3 (NC)
- net BUCK_VCC: no longer names the net of C8.1, U1.5 (VCC)
- net CAN_STB: no longer names the net of R43.1, U6.8 (STBY)
- net CAN_TERM: no longer names the net of JP1.2 (B), R25.1
- net ETH_LED_G_A: no longer names the net of J6.9, R41.2
- net ETH_LED_Y_A: no longer names the net of J6.12, R42.2
- net ETH_RCT: no longer names the net of C19.1, J6.5 (RCT)
- net ETH_RXB: no longer names the net of C17.1, R22.2, R23.2
- net ETH_SHIELD: no longer names the net of C20.1, J6.SH
- net ETH_TCT: no longer names the net of C18.1, J6.4 (TCT), R24.2
- net GPIO22: no longer names the net of TP3.1, U4.20 (GPIO22)
- net GPIO23: no longer names the net of TP4.1, U4.21 (GPIO23)
- net GPIO4: no longer names the net of TP1.1, U4.4 (MTMS/GPIO4/ADC1_CH4)
- net GPIO5: no longer names the net of TP2.1, U4.5 (MTDI/GPIO5/ADC1_CH5)
- net J5_VREF: no longer names the net of J5.1 (Pin_1), R33.2
- net LED_PWR: no longer names the net of D5.2 (A), R44.2
- net RGB_DIN: no longer names the net of D6.4 (DIN), R31.2, R32.2
- net RGB_DIN_5V: no longer names the net of R31.1, U9.4
- net RGB_HCT_MID: no longer names the net of U9.2, U9.3
- net SPI_SCLK_C6: no longer names the net of R19.1, U4.6 (MTCK/GPIO6/ADC1_CH6)
- net U0TXD_C6: no longer names the net of R39.1, U4.25 (U0TXD/GPIO16)
- net USB_CC1: no longer names the net of J4.A5 (CC1), R28.1
- net USB_CC2: no longer names the net of J4.B5 (CC2), R29.1
- net VBUS_EN_IN: no longer names the net of D9.2 (A), R10.2, R11.1, U3.3 (EN)
- net VBUS_ILIM: no longer names the net of R12.1, U3.5 (ILIM)
- net W_1V2O: no longer names the net of C30.1, U5.22 (1V2O)
- net W_EXRES: no longer names the net of R40.1, U5.10 (EXRES1)
- net W_TOCAP: no longer names the net of C29.1, U5.20 (TOCAP)
- net XTAL25_I: no longer names the net of C40.1, U5.30 (XI/CLKIN), Y1.1
- net XTAL25_O: no longer names the net of C41.1, U5.31 (XO), Y1.3
Other:
- note added: "1. TÁP: +24V_IN → F1 → D1 → +24V_P → D8 → VIN_BUCK (U1 LMR36015 → 3,3 V); +24V_P → R7 → +24V_F → U2 P78E05 → +5V"
- note added: "2. V_BUS – U3 TPS2553: EN-osztó a +24V_P-ről (csak 24 V mellett BE); a GPIO20 a D9-en (BAT54) át letiltja (D61); korlát 382/425/476 mA"
- note added: "3,3 V – U1 LMR36015BRNXR (1 MHz, L1 6,8 µH): a FOOTPRINT a TI Ultra Librarian-ből!"
- note added: "3. ESP32-C6-WROOM-1-N16 (fém szekrénybe -1U ugyanerre a footprintre, D63) – strapping: GPIO8 = 1, GPIO9 = 1 (BOOT gomb → 0), GPIO15"
- note added: "4. ETHERNET – U5 W5500 + J6 HR911105A MagJack (opcionálisan beültetve; MDI a WIZnet use_mag referencia szerint)"
- note added: "5. USB-C – csak eszköz, csak táp-fogyasztó"
- note added: "6. CAN – U6 TCAN1044AVDRQ1 (MCP2562 szimbólum, lábról lábra azonos) · JP2 alap 5 V: 1044/2562 · 3V3: 330/230 (D60)"
- note added: "7. GOMBOK, LED-EK, RGB, DEBUG – U9 és R32 egyszerre NE legyen beültetve"
- note added: "CC1/CC2 külön 5,1 kΩ; USBLC6 az aljzatnál, 22 Ω a C6-nál"
- note added: "ESD (U7) · lezárás: JP1 + R25 (csak a lánc végén)"
- note added: "Generálva (hardware/gen/vezerlo.py) – a VEZERLO-SPEC.md alapján; kézi szerkesztés helyett a generátort módosítsd."
- note added: "J5: 1 VREF · 2 GND · 3 TX · 4 RX · 5 EN · 6 BOOT"
- note added: "MDI-lezárás: TX 49,9 Ω a +3V3A-ra (TXB), RX 49,9 Ω a RXB-re; a RXB csak C17-en át a GND-re"
- note added: "RGB_DIN"
- note added: "USB csak a 3,3 V-os buckot táplálja (D3) – a V_BUS USB-ről hardveresen KI (D61); D57: a C1 elkó kötelező, a 24 V-os tápot ≤ 26 V-ra"
- note added: "VBUS_SENSE: 5 V → 0,9 V (GPIO1)"
- note added: "W5500 hidegítés: AVDD-lábanként 100 nF; FB1 = HH-1M1608-121JT, ≥ 300 mA"
- note added: "felhúzások (10 k): GPIO8 · BOOT · CS · RST · GPIO15 · CAN_TX"
- note removed: "2.1 BEMENET: +24V_IN → F1 → D1 → +24V_P; USB csak a 3,3 V-os buckot táplálja (D3) – a V_BUS USB-ről hardveresen KI (D61)"
- note removed: "2.2 3,3 V – LMR36015BRNXR (1 MHz): FOOTPRINT a TI Ultra Librarian-ből!"
- note removed: "2.4 V_BUS – TPS2553: EN osztó a +24V_P-ről (csak 24 V mellett BE), GPIO20 BAT54-en át letiltja"
- note removed: "3. ESP32-C6-WROOM-1-N16 (fém szekrénybe -1U – az EPAD helyét ellenőrizni!)"
- note removed: "4. ETHERNET – W5500 + HR911105A MagJack (opcionálisan beültetve; MDI a WIZnet use_mag referencia szerint)"
- note removed: "5–6. CAN – TCAN1044AVDRQ1 (MCP2562 szimbólum, lábról lábra azonos) · JP2 alap 5V: 1044/2562 · 3V3: 330/230"
- note removed: "7. USB-C – csak eszköz, csak táp-fogyasztó (CC1/CC2 külön 5,1 kΩ)"
- note removed: "8. GOMBOK, LED-EK, DEBUG – U9 és R32 egyszerre NE legyen beültetve"
- note removed: "VÁZLAT – generálva a VEZERLO-SPEC.md alapján (2026-10-14). Elrendezést rendezd; a bekötés címkékkel kész."

Commit message: Hardver: átnézés (C320 javítva), LoRa-előkészítés (D68), bővítők (D69), R6/R7 = 0 Ω (D70)
- bemeneti modul: a HDC3020 hidegítője C330 lett (a C320 kétszer szerepelt);
  a generátor mostantól hibát dob duplikált jelölésre
- vezérlő: E22-900M22S LoRa + u.FL + 74LVC1G04, minden DNP; J8 bővítő (GPIO5),
  7 mérőpont; spec szerinti DNP-k (USB C, 1 MΩ, PMODE, CAN-fojtó + áthidalók);
  saját footprint az LMR36015-höz (RNX) és az E22-höz
- modulmag: HW_REV osztó (PB0), DNP J4 2 × 5 bővítő; relé: DNP SCT-013 → PA0
- mind az öt lap vizuálisan rendbe téve; R6/R7 = 0 Ω
- specek és döntésnapló frissítve (D68–D70)

Co-Authored-By: Claude Opus 5.5 <noreply@anthropic.com>
Parts:
- added C49, C50: DNP, Capacitor_SMD:C_0603_1608Metric, symbol Device:C
- added C51: 10µ, Capacitor_SMD:C_0805_2012Metric, symbol Device:C
- added C52: 100n, Capacitor_SMD:C_0603_1608Metric, symbol Device:C
- added J7: u.FL, Connector_Coaxial:U.FL_Hirose_U.FL-R-SMT-1_Vertical, symbol Connector:Conn_Coaxial
- added J8: BŐVÍTŐ, Connector_JST:JST_PH_B3B-PH-K_1x03_P2.00mm_Vertical, symbol Connector_Generic:Conn_01x03
- added JP4, JP5: áthidaló, Jumper:SolderJumper-2_P1.3mm_Bridged_RoundedPad1.0x1.5mm, symbol Jumper:SolderJumper_2_Bridged
- added L2: DNP, Inductor_SMD:L_CommonModeChoke_Coilank_ACM3225, symbol Device:Filter_EMI_CommonMode
- added R46: 0R, Resistor_SMD:R_0603_1608Metric, symbol Device:R
- added R47: 1M, Resistor_SMD:R_0603_1608Metric, symbol Device:R
- added R48, R49, R50, R53: DNP, Resistor_SMD:R_0603_1608Metric, symbol Device:R
- added R51: 10k, Resistor_SMD:R_0603_1608Metric, symbol Device:R
- added R52: 4k7, Resistor_SMD:R_0603_1608Metric, symbol Device:R
- added TP5: CAN_H, TestPoint:TestPoint_Pad_D1.5mm, symbol Connector:TestPoint
- added TP6: CAN_L, TestPoint:TestPoint_Pad_D1.5mm, symbol Connector:TestPoint
- added TP7: GND, TestPoint:TestPoint_Pad_D1.5mm, symbol Connector:TestPoint
- added U10: E22-900M22S, modularis:Ebyte_E22-900M22S, symbol modularis:E22-900M22S
- added U11: 74LVC1G04, Package_TO_SOT_SMD:SOT-353_SC-70-5, symbol 74xGxx:74LVC1G04
- R7: value 10R -> 0R; Megjegyzés impulzusbíró, 2512; 0 Ω-mal áthidalható (D57) -> D70: 0 Ω; a footprint marad – szükség esetén 10 Ω impulzusb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
- TP1: value GPIO4 -> +24V_P
- TP2: value GPIO5 -> +5V
- TP3: value GPIO22 -> +3V3
- TP4: value GPIO23 -> V_BUS
- U1: footprint (none) -> modularis:TI_VQFN-HR-12_RNX0012B
Connections:
- net +24V_P: now also TP1.1
- net +3V3: now also TP3.1, J8.1 (Pin_1), R46.1, R51.1, R52.1
- net +5V: now also TP2.1
- net CAN_H: now also JP4.2 (B), L2.2, TP5.1; no longer U6.7 (CANH)
- net CAN_L: now also JP5.2 (B), L2.4, TP6.1; no longer U6.6 (CANL)
- net GND: now also C49.2, C50.2, C51.2, C52.2, J7.2 (Ext), J8.3 (Pin_3), R48.2, R49.2, R50.2, R53.2, TP7.1, U10.1 (GND), U10.10 (GND), U10.11 (GND), U10.12 (GND), U10.2 (GND), U10.20 (GND), U10.22 (GND), U10.3 (GND), U10.4 (GND), U10.5 (GND), U11.3 (GND)
- net SPI_MISO: now also U10.16 (MISO)
- net SPI_MOSI: now also U10.17 (MOSI)
- net SPI_SCLK: now also U10.18 (SCK)
- net USB_DM: now also C50.1
- net USB_DP: now also C49.1
- net V_BUS: now also TP4.1
- net W5500_RST: now also U10.15 (NRST)
- net at C41.1, U5.31 (XO), Y1.3: now also R47.2
- net LORA_CS: now reaches U4.20 (GPIO22)
- net LORA_CS: now also R51.2, U10.19 (NSS); no longer TP3.1
- net at C40.1, U5.30 (XI/CLKIN), Y1.1: now also R47.1
- net PMODE2: now reaches U5.43 (PMODE2)
- net PMODE2: now also R50.1
- net PMODE1: now reaches U5.44 (PMODE1)
- net PMODE1: now also R49.1
- net PMODE0: now reaches U5.45 (PMODE0)
- net PMODE0: now also R48.1
- net LORA_BUSY: now reaches U4.21 (GPIO23)
- net LORA_BUSY: now also U10.14 (BUSY); no longer TP4.1
- net EXP_GPIO5: now reaches U4.5 (MTDI/GPIO5/ADC1_CH5)
- net EXP_GPIO5: now also J8.2 (Pin_2), R52.2, R53.1; no longer TP2.1
- net LORA_DIO1: now reaches U4.4 (MTMS/GPIO4/ADC1_CH4)
- net LORA_DIO1: now also U10.13 (DIO1); no longer TP1.1
- new net: J7.1 (In), U10.21 (ANT)
- new net +3V3_LORA: C51.1, C52.1, R46.2, U10.9 (VCC), U11.5 (VCC)
- new net CAN_H_T: JP4.1 (A), L2.1, U6.7 (CANH)
- new net CAN_L_T: JP5.1 (A), L2.3, U6.6 (CANL)
- new net LORA_DIO2: U10.7 (TXEN), U10.8 (DIO2), U11.2
- new net LORA_RXEN: U10.6 (RXEN), U11.4
- no-connect marks 25 -> 23
Other:
- note added: "3,3 V – U1 LMR36015BRNXR (1 MHz, L1 6,8 µH), VQFN-HR (RNX0012B)"
- note added: "8. LoRa (D68) – U10 Ebyte E22-900M22S (SX1262, 868 MHz) + J7 u.FL – MINDEN DNP, később beültethető"
- note added: "9. BŐVÍTŐ (J8, GPIO5 = ADC1_CH5): 1-wire / gomb / revízió-osztó · MÉRŐPONTOK"
- note added: "CAN-fojtó: L2 DNP + JP4/JP5 zárva; fojtóval: JP4/JP5 átvágva"
- note added: "SPI a W5500-zal közös; NRST = W5500_RST (közös reset); TXEN = DIO2, RXEN = ¬DIO2 (U11) → firmware: setDio2AsRfSwitch"
- note added: "VBG (18) NYITVA · RSVD 38–42 NYITVA · RSVD 23 GND · PMODE nyitva = auto-negotiation (R48–R50 lehúzás DNP)"
- note added: "W5500 PMODE-lehúzás (DNP)"
- note removed: "3,3 V – U1 LMR36015BRNXR (1 MHz, L1 6,8 µH): a FOOTPRINT a TI Ultra Librarian-ből!"
- note removed: "VBG (18) NYITVA · RSVD 38–42 NYITVA · RSVD 23 GND · PMODE nyitva (auto-negotiation)"

Commit message: Hardver: központi 5 V, közös föld, 12–26 V, HW-ID 16 sáv (D71)
Vezérlő: LMR33630 (5,2 V) + LM66200 (USB-vel VAGY-olva) + TPS259531 eFuse (2 A);
F1 2 A, D1 B360 a 12 V-os működéshez. Modulmag: táp a buszról (AP2112K), TCAN1044AV,
nincs izoláció, PC1 = VBUS_SENSE. LED/relé: VIN_SENSE a PB11-en, relémodul saját
tekercs-táppal. Bemeneti modul: nincs 24 V. HW-ID/HW_REV 16 sáv. Specifikációk,
áttekintés, beszerzés, ütemterv frissítve.

Co-Authored-By: Claude Opus 5.5 <noreply@anthropic.com>
Parts:
- removed U2: P78E05-1000, Converter_DCDC:Converter_DCDC_RECOM_R-78E-0.5_THT, symbol Converter_DCDC:R-78E5.0-1.0
- removed U3: TPS2553DBVR, Package_TO_SOT_SMD:SOT-23-6, symbol modularis:TPS2553DBV
- added C53: 220n/50V, Capacitor_SMD:C_0603_1608Metric, symbol Device:C
- added C54: 1µ/16V, Capacitor_SMD:C_0603_1608Metric, symbol Device:C
- added C55: 100n, Capacitor_SMD:C_0603_1608Metric, symbol Device:C
- added C56, C57, C58, C59: 22µ, Capacitor_SMD:C_1206_3216Metric, symbol Device:C
- added C60: 22n, Capacitor_SMD:C_0603_1608Metric, symbol Device:C
- added L3: 8,2µH, Inductor_SMD:L_Bourns_SRN6045TA, symbol Device:L
- added R54: 100k 1%, Resistor_SMD:R_0603_1608Metric, symbol Device:R
- added R55: 23,7k 1%, Resistor_SMD:R_0603_1608Metric, symbol Device:R
- added U12: LM66200DRLR, Package_TO_SOT_SMD:SOT-583-8, symbol modularis:LM66200DRL
- added U2: LMR33630ADDA, Package_SO:Texas_HSOP-8-1EP_3.9x4.9mm_P1.27mm_ThermalVias, symbol Regulator_Switching:LMR33630ADDA
- added U3: TPS259531DSGR, Package_SON:Texas_DSG0008A_WSON-8-1EP_2x2mm_P0.5mm_EP0.9x1.6mm, symbol modularis:TPS259531DSG
- C10, C11, C12: value 22µ/10V -> 22µ; Megjegyzés (none) -> X7R, 10 V, 1206
- C2: Megjegyzés (none) -> CIN az U2 VIN-lábánál; mellette C53 220 nF
- D1: value SS16 -> B360; footprint Diode_SMD:D_SMA -> Diode_SMD:D_SMC; Megjegyzés (none) -> 60 V, 3 A – D71: a bemeneti áram 12 V-on ~1,2 A
- F1: value 1A -> 2A; Megjegyzés ≥ 32 V, gyors -> ≥ 32 V, gyors; D71: 12 V-on és 2 A-es buszterhelésnél ~1,2 A
- R10: value 470k -> 100k
- R12: value 61,9k 1% -> 1,02k 1%; Megjegyzés → 382/425/476 mA -> R = 2000 / (I − 0,04) → 2,0 A
- R34: Megjegyzés FAULT felhúzás (nyitott drain) -> FLT felhúzás (nyitott drain)
Connections:
- net +24V_F: now also C53.1, U2.2 (VIN), U2.3 (EN)
- net +24V_P: no longer R10.1
- net +5V: now also R10.1, U12.2 (VOUT), U12.7 (VOUT), U3.3 (IN), U3.4 (IN)
- net GND: now also C53.2, C54.2, C56.2, C57.2, C58.2, C59.2, C60.2, R55.2, U12.1 (GND), U12.4 (~{ON}), U12.5 (GND), U2.1 (GND), U2.9 (GND), U3.8 (GND), U3.9 (PAD)
- net VBUS_FAULT: now also U3.6 (~{FLT})
- net VUSB: now also U12.6 (VIN2)
- net V_BUS: now also U3.5 (OUT)
- net at D9.2 (A), R10.2, R11.1: now also U3.2 (EN/UVLO)
- net at R12.1: now also U3.7 (ILM)
- new net: C54.1, U2.6 (VCC)
- new net: C55.2, L3.1, U2.8 (SW)
- new net: C60.1, U3.1 (dVdt)
- new net: R54.2, R55.1, U2.5 (FB)
- new net: C55.1, U2.7 (BOOT)
- new net +5V_BUCK: C56.1, C57.1, C58.1, C59.1, L3.2, R54.1, U12.3 (VIN1)
- no-connect marks 23 -> 25
Other:
- note added: "1. TÁP (12–26 V): +24V_IN → F1 → D1 → +24V_P → D8 → VIN_BUCK (U1 LMR36015 → 3,3 V); +24V_P → R7 → +24V_F → U2 LMR33630 (5,2 V) → U12 LM66200 → +5V"
- note added: "2. V_BUS – U3 TPS259531 eFuse (D71): 2 A-es korlát, 5,7 V-os túlfeszültség-vágás; EN-osztó a +5V-ról (bármelyik forrásról BE), a GPIO20 a D9-en (BAT54) át letiltja"
- note added: "D71: központi 5 V a buszra (2 A); USB-ről is: az U12 a nagyobbat választja (buck 5,2 V > USB). D57: a C1 elkó kötelező; a tápot ≤ 26 V-ra (az U2 max. 36 V)"
- note removed: "1. TÁP: +24V_IN → F1 → D1 → +24V_P → D8 → VIN_BUCK (U1 LMR36015 → 3,3 V); +24V_P → R7 → +24V_F → U2 P78E05 → +5V"
- note removed: "2. V_BUS – U3 TPS2553: EN-osztó a +24V_P-ről (csak 24 V mellett BE); a GPIO20 a D9-en (BAT54) át letiltja (D61); korlát 382/425/476 mA"
- note removed: "USB csak a 3,3 V-os buckot táplálja (D3) – a V_BUS USB-ről hardveresen KI (D61); D57: a C1 elkó kötelező, a 24 V-os tápot ≤ 26 V-ra"

Commit message: Hardver: footprintek a gyártói rajzokkal ellenőrizve, W5500 MDI a WIZnet-referencia szerint (D72)
E22 padok ±7,0 mm-re (két referencia-footprinttel egyezik), TPS2595 ThermalVias,
LMR36015 RNX és LM66200 DRL összevetve. W5500 RX: soros 6,8 nF, a lezárás közepe
az RCT-re + 10 nF, a MagJack 8-as lába és árnyékolása ETH_CGND (1 nF / 2 kV).

Co-Authored-By: Claude Opus 5.5 <noreply@anthropic.com>
Parts:
- added C61: 6,8n, Capacitor_SMD:C_0603_1608Metric, symbol Device:C
- C17: value 6,8n -> 10n; Megjegyzés a RXB csak kondenzátoron át a GND-re, NEM a 3,3 V-ra -> a WIZnet-referencia C15-je: az RX-lezárás közepe és az RCT,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
- C19: Megjegyzés (none) -> soros, a W5500 RX-lába és a MagJack között
- C20: Megjegyzés (none) -> WIZnet-referencia C16: a MagJack árnyékolása és a Bob Smith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
- R20, R21, R22, R23: value 49,9R 1% -> 49R9; Megjegyzés (none) -> 1 %
- U3: footprint Package_SON:Texas_DSG0008A_WSON-8-1EP_2x2mm_P0.5mm_EP0.9x1.6mm -> Package_SON:Texas_DSG0008A_WSON-8-1EP_2x2mm_P0.5mm_EP0.9x1.6mm_ThermalVias
Connections:
- net ETH_RXN: now also C61.2; no longer R23.1, U5.5 (RXN)
- net ETH_RXP: now also C19.2; no longer R22.1, U5.6 (RXP)
- net GND: no longer C19.2, J6.8
- net ETH_RCT: now reaches C17.1, R22.2, R23.2
- net ETH_RCT: now also J6.5 (RCT)
- net ETH_RXP_W: now reaches C19.1
- net ETH_RXP_W: now also R22.1, U5.6 (RXP); no longer J6.5 (RCT)
- net ETH_CGND: now reaches C20.1, J6.SH
- net ETH_CGND: now also J6.8
- new net ETH_RXN_W: C61.1, R23.1, U5.5 (RXN)
Other:
- note added: "MDI (WIZnet-referencia): TX 49,9 Ω a +3V3A-ra; RX 49,9 Ω → RCT + 10 nF; RX-ben soros 6,8 nF"
- note removed: "MDI-lezárás: TX 49,9 Ω a +3V3A-ra (TXB), RX 49,9 Ω a RXB-re; a RXB csak C17-en át a GND-re"
