File: hardware/vezerlo/vezerlo.kicad_sch (KiCad schematic)
At the start: 158 parts, among them J1 24V IN, J2 BUS (XH), J3 BUS (XH), J4 USB-C 16P, J5 DEBUG, J6 HR911105A, J7 u.FL, J8 BŐVÍTŐ, SW1 RESET, SW2 BOOT, U1 LMR36015BRNXR, U10 E22-900M22S, U11 74LVC1G04, U12 LM66200DRLR, U2 LMR33630ADDA, U3 TPS259531DSGR, U4 ESP32-C6-WROOM-1-N16, U5 W5500, U6 TCAN1044AVDRQ1, U7 ESD2CAN24-Q1, U8 USBLC6-2SC6, U9 74HCT14D, Y1 25MHz ±30ppm

Commit message: Hardver: szakértői javítások (D74–D77), STM32L433 + SN65HVD230 + GND-ági polaritásvédelem (D78–D81), teljes ellenőrzés
- D74–D77: busz-GND ellenállás, CAN-fojtó-hely, TVS a +5V_BUCK-on és a VUSB-n, bemenetvédelem,
  230 V-os és antenna-tiltás a NYÁK-on, SCT-jack footprint
- D78–D80: modul-MCU STM32L433RCT3 (VIN_SENSE PB1, LED: TIM15/TIM16, I_SENSE PA3), modul-transceiver
  SN65HVD230, N-FET a GND-ágban (vezérlő Q1, LED Q201, relé Q100), MCP9701A, táp-LED a +5V-ról,
  2 oz a LED-/relémodulon, AP2112K marad; D81 javaslat (TPD4E02B04 a bemeneteken)
- CubeMX-projektek L433-ra, fejsoros kódgenerálással ellenőrizve (minden periféria inicializálódik)
- gen/ellenorzes.py (ERC, láb ↔ pad, modulmag, CubeMX, polaritásvédelem, NYÁK ↔ rajz, DRC) – 0 hiba
- gen/bom.sh + bom/*.csv darabjegyzék; docs/komponenslista.md a konzulensnek
- kontextus: DONTESEK D74–D81, specifikációk, ATTEKINTES, NAPLO, beszerzési lista; alkatrészkészlet-jegyzet (claude.ai)

Co-Authored-By: Claude Opus 5.5 <noreply@anthropic.com>
Parts:
- removed D1: B360, Diode_SMD:D_SMC, symbol Device:D_Schottky
- added D10: SMBJ6.0A, Diode_SMD:D_SMB, symbol Device:D_Zener
- added D11: SMF5.0A, Diode_SMD:D_SOD-123F, symbol Device:D_Zener
- added D12: BZT52C15, Diode_SMD:D_SOD-123, symbol Device:D_Zener
- added Q1: IRFR1205, Package_TO_SOT_SMD:TO-252-2, symbol Transistor_FET:Q_NMOS_GDS
- added R56: 10k, Resistor_SMD:R_0603_1608Metric, symbol Device:R
- R44: Megjegyzés (none) -> D78: a +5V-ról – a zöld LED (522 nm) nyitófeszültsége ~3 V
- U10: Megjegyzés Ebyte E22-900M22S, 14 × 20 mm; az antennarész alatt réz-tiltás -> Ebyte E22-900M22S, 14 × 20 mm; az antennarész alatt réz-tiltás. EU 868 MHz (ERC/REC 70-03): 25 mW ERP / 14 dBm, kitöltés 1 %; a 22 dBm csak a 869,4–869,65 MHz-es sávban (≤ 500 mW, 10 %) – a firmware korlátozza (D77)
Connections:
- net +24V_P: now also F1.2, R56.1
- net +3V3: no longer R44.1
- net +5V: now also R44.1
- net +5V_BUCK: now also D10.1 (K)
- net GND: now also D10.2 (A), D11.2 (A), D12.2 (A), Q1.3 (S); no longer J1.2 (Pin_2)
- net VUSB: now also D11.1 (K)
- new net: D12.1 (K), Q1.1 (G), R56.2
- new net GND_IN: J1.2 (Pin_2), Q1.2 (D)
Other:
- note added: "1. TÁP (12–26 V): +24V_IN → F1 → +24V_P (Q1 a GND-ágban, D78) → D8 → VIN_BUCK (U1 LMR36015 → 3,3 V); +24V_P → R7 → +24V_F → U2 LMR33630 (5,2 V) → U12 LM66200 → +5V"
- note removed: "1. TÁP (12–26 V): +24V_IN → F1 → D1 → +24V_P → D8 → VIN_BUCK (U1 LMR36015 → 3,3 V); +24V_P → R7 → +24V_F → U2 LMR33630 (5,2 V) → U12 LM66200 → +5V"
