File: hardware/vezerlo/vezerlo.kicad_sch (KiCad schematic)
At the start: 162 parts, among them J1 24V IN, J2 BUS (XH), J3 BUS (XH), J4 USB-C 16P, J5 DEBUG, J6 HR911105A, J7 u.FL, J8 BŐVÍTŐ, Q1 IRFR1205, SW1 RESET, SW2 BOOT, U1 LMR36015BRNXR, U10 E22-900M22S, U11 74LVC1G04, U12 LM66200DRLR, U2 LMR33630ADDA, U3 TPS259531DSGR, U4 ESP32-C6-WROOM-1-N16, U5 W5500, U6 TCAN1044AVDRQ1, U7 ESD2CAN24-Q1, U8 USBLC6-2SC6, U9 74HCT14D, Y1 25MHz ±30ppm

Commit message: Hardver: legolcsóbb beszerzés (D84) – Hestore + DigiKey, a rajz a kapható típusokra igazítva; beszerzési lista
- gen/beszerzes.py → bom/beszerzes.csv: BOM-tételenként forrás, Hestore-kód, nettó ár, készlet
- J1/J100 Degson DG250, J201 DG128 (15 A), J202–J204 KF128, F201 15 A; L1/L3 HPI0630 (saját footprint);
  R209 CRE2512; C40/C41 12 pF; ESP32-C6-WROOM-1-N8; SS56C, BAT54HT1G, STPS3L60U, BLM18EG221
- NYÁK-ok újragenerálva (a layout még nem indult el); bekötés változatlan, ellenorzes.py: 0 hiba
- SAMPLE-KERESEK: az NTMFS5C604NL nincs kézben (javítva)

Co-Authored-By: Claude Opus 5.5 <noreply@anthropic.com>
Claude-Session: https://claude.ai/code/session_01KVtZMUPbtveTXy9VyJshyt
Parts:
- C4: value 4µ7/50V -> 10µ/50V
- C40: value 18p -> 12p; Megjegyzés C = 2 × (CL − 3…5 pF) a megvett kvarcból -> C = 2 × (CL − 3…5 pF); a CX3225 CL-je 10 pF → 12 pF (D84)
- C41: value 18p -> 12p
- C9: value 20p -> 22p; Megjegyzés CFF, R3-mal párhuzamosan -> CFF, R3-mal párhuzamosan (20 pF helyett a kapható 22 pF – D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
- D3: value B360 -> SS56C; Megjegyzés 60 V-os kell (túlfeszültségnél VIN_BUCK ~45 V, VUSB ~0 V) -> 60 V-os kell (túlfeszültségnél VIN_BUCK ~45 V, VUSB ~0 V); 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
- D9: value BAT54WS -> BAT54HT1G
- FB1: value 120R@100MHz -> BLM18EG221; Megjegyzés HH-1M1608-121JT, ≥ 300 mA -> D84: Murata BLM18EG221TN1D – 220 Ω @ 100 MHz, 1 A, 0,15 Ω
- J1: footprint TerminalBlock_Phoenix:TerminalBlock_Phoenix_PT-1,5-2-3.5-H_1x02_P3.50mm_Horizontal -> TerminalBlock_Degson:TerminalBlock_Degson_DG250-3.5-02P_1x02_P3.50mm_45Degree; Megjegyzés push-in sorkapocs – a típus a DIN-ház vállához (D50) -> D84: Degson DG250-3.5-02P – rugós, nyomógombos, 8 A (UL), 0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
- L1: footprint Inductor_SMD:L_Coilcraft_XAL5030-XXX -> modularis:L_FerroCore_HPI0630; Megjegyzés árnyékolt, Isat ≥ 2,1 A (ideálisan ≥ 2,8 A), ~5 × 5 mm -> D84: HPI0630-6R8 – árnyékolt, Isat 4,9 A, 53 mΩ
- L3: footprint Inductor_SMD:L_Bourns_SRN6045TA -> modularis:L_FerroCore_HPI0630; Megjegyzés árnyékolt, Isat ≥ 3,5 A, ~14 mΩ (pl. SRN6045TA-8R2M) – 3 A-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 -> D84: HPI0630-8R2 – árnyékolt, Isat 3,8 A, 59,5 mΩ (2 A-en ~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
- U4: value ESP32-C6-WROOM-1-N16 -> ESP32-C6-WROOM-1-N8
- Y1: Megjegyzés (none) -> D84: Kyocera CX3225FB25000F0FZZH1 – ±20 ppm, CL = 10 pF (He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
Other:
- note added: "3. ESP32-C6-WROOM-1-N8 (D84; fém szekrénybe -1U ugyanerre a footprintre, D63) – strapping: GPIO8 = 1, GPIO9 = 1 (BOOT gomb → 0), GPIO15"
- note added: "W5500 hidegítés: AVDD-lábanként 100 nF; FB1 = BLM18EG221TN1D, 1 A (D84)"
- note removed: "3. ESP32-C6-WROOM-1-N16 (fém szekrénybe -1U ugyanerre a footprintre, D63) – strapping: GPIO8 = 1, GPIO9 = 1 (BOOT gomb → 0), GPIO15"
- note removed: "W5500 hidegítés: AVDD-lábanként 100 nF; FB1 = HH-1M1608-121JT, ≥ 300 mA"
Changed lines of the file:
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@@
 		)
 	)
-	(text "W5500 hidegítés: AVDD-lábanként 100 nF; FB1 = HH-1M1608-121JT, ≥ 300 mA"
+	(text "W5500 hidegítés: AVDD-lábanként 100 nF; FB1 = BLM18EG221TN1D, 1 A (D84)"
 		(exclude_from_sim no)
 		(at 300 287.18 0)
@@
 		)
 	)
-	(text "3. ESP32-C6-WROOM-1-N16 (fém szekrénybe -1U ugyanerre a footprintre, D63) – strapping: GPIO8 = 1, GPIO9 = 1 (BOOT gomb → 0), GPIO15"
+	(text "3. ESP32-C6-WROOM-1-N8 (D84; fém szekrénybe -1U ugyanerre a footprintre, D63) – strapping: GPIO8 = 1, GPIO9 = 1 (BOOT gomb → 0), GPIO15"
 		(exclude_from_sim no)
 		(at 20 166 0)
@@
 			)
 		)
-		(property "Value" "120R@100MHz"
+		(property "Value" "BLM18EG221"
 			(at 330.2 299.72 90)
 			(show_name no)
@@
 			)
 		)
-		(property "Megjegyzés" "HH-1M1608-121JT, ≥ 300 mA"
+		(property "Megjegyzés" "D84: Murata BLM18EG221TN1D – 220 Ω @ 100 MHz, 1 A, 0,15 Ω"
 			(at 330.2 297.18 90)
 			(hide yes)
@@
 			)
 		)
-		(property "Value" "B360"
+		(property "Value" "SS56C"
 			(at 110.49 345.44 0)
 			(show_name no)
@@
 			)
 		)
-		(property "Megjegyzés" "60 V-os kell (túlfeszültségnél VIN_BUCK ~45 V, VUSB ~0 V)"
+		(property "Megjegyzés" "60 V-os kell (túlfeszültségnél VIN_BUCK ~45 V, VUSB ~0 V); SS56C: 60 V, 5 A, SMC (D84)"
 			(at 110.49 342.9 0)
 			(hide yes)
@@
 			)
 		)
-		(property "Value" "18p"
+		(property "Value" "12p"
 			(at 318.77 243.84 90)
 			(show_name no)
@@
 			)
 		)
-		(property "Footprint" "TerminalBlock_Phoenix:TerminalBlock_Phoenix_PT-1,5-2-3.5-H_1x02_P3.50mm_Horizontal"
+		(property "Footprint" "TerminalBlock_Degson:TerminalBlock_Degson_DG250-3.5-02P_1x02_P3.50mm_45Degree"
 			(at 27.94 55.88 0)
 			(hide yes)
@@
 			)
 		)
-		(property "Megjegyzés" "push-in sorkapocs – a típus a DIN-ház vállához (D50)"
+		(property "Megjegyzés" "D84: Degson DG250-3.5-02P – rugós, nyomógombos, 8 A (UL), 0,2–1,5 mm²; Hestore 100.441.02"
 			(at 27.94 55.88 0)
 			(hide yes)
@@
 			)
 		)
-		(property "Value" "ESP32-C6-WROOM-1-N16"
+		(property "Value" "ESP32-C6-WROOM-1-N8"
 			(at 106.68 198.12 0)
 			(show_name no)
@@
 			)
 		)
+		(property "Megjegyzés" "D84: Kyocera CX3225FB25000F0FZZH1 – ±20 ppm, CL = 10 pF (Hestore 100.494.61)"
+			(at 330.2 237.49 90)
+			(hide yes)
+			(show_name no)
+			(do_not_autoplace no)
+			(effects
+				(font
+					(size 1.27 1.27)
+				)
+			)
+		)
 		(pin "1"
 		)
@@
 			)
 		)
-		(property "Footprint" "Inductor_SMD:L_Bourns_SRN6045TA"
+		(property "Footprint" "modularis:L_FerroCore_HPI0630"
 			(at 240.03 48.26 90)
 			(hide yes)
@@
 			)
 		)
-		(property "Megjegyzés" "árnyékolt, Isat ≥ 3,5 A, ~14 mΩ (pl. SRN6045TA-8R2M) – 3 A-ig"
+		(property "Megjegyzés" "D84: HPI0630-8R2 – árnyékolt, Isat 3,8 A, 59,5 mΩ (2 A-en ~0,24 W)"
 			(at 240.03 48.26 90)
 			(hide yes)
@@
 			)
 		)
-		(property "Value" "18p"
+		(property "Value" "12p"
 			(at 318.77 236.22 90)
 			(show_name no)
@@
 			)
 		)
-		(property "Megjegyzés" "C = 2 × (CL − 3…5 pF) a megvett kvarcból"
+		(property "Megjegyzés" "C = 2 × (CL − 3…5 pF); a CX3225 CL-je 10 pF → 12 pF (D84)"
 			(at 318.77 233.68 90)
 			(hide yes)
@@
 			)
 		)
-		(property "Value" "4µ7/50V"
+		(property "Value" "10µ/50V"
 			(at 60.96 109.22 0)
 			(show_name no)
@@
 			)
 		)
-		(property "Value" "BAT54WS"
+		(property "Value" "BAT54HT1G"
 			(at 361.95 147.32 90)
 			(show_name no)
@@
 			)
 		)
-		(property "Footprint" "Inductor_SMD:L_Coilcraft_XAL5030-XXX"
+		(property "Footprint" "modularis:L_FerroCore_HPI0630"
 			(at 128.27 114.3 90)
 			(hide yes)
@@
 			)
 		)
-		(property "Megjegyzés" "árnyékolt, Isat ≥ 2,1 A (ideálisan ≥ 2,8 A), ~5 × 5 mm"
+		(property "Megjegyzés" "D84: HPI0630-6R8 – árnyékolt, Isat 4,9 A, 53 mΩ"
 			(at 128.27 114.3 90)
 			(hide yes)
@@
 			)
 		)
-		(property "Value" "20p"
+		(property "Value" "22p"
 			(at 149.86 121.92 0)
 			(show_name no)
@@
 			)
 		)
-		(property "Megjegyzés" "CFF, R3-mal párhuzamosan"
+		(property "Megjegyzés" "CFF, R3-mal párhuzamosan (20 pF helyett a kapható 22 pF – D84)"
 			(at 147.32 120.65 0)
 			(hide yes)

Commit message: Hardver: legolcsóbb beszerzés LCSC-ről (D85), megszűnt FET-ek pótlása, LCSC-kosárlista
- gen/lcsc.py: LCSC-árak a JLC alkatrészkeresőjéből; gen/beszerzes.py soronként a legolcsóbb forrás (Hestore / LCSC, ÁFA-val)
- bom/lcsc-kosar.csv: 99 tétel (~15 eFt), az LCSC BOM Tooljába feltölthető; házak később, ST-Link/Nucleo kézben
- Q202–Q207 NTD5C648NL → NCE6080K, Q201 NTMFS5C604NL → NCEP6090AGU (nem kaphatók), F201 → NANO² 15 A,
  D211–D216 SS56B, J1/J100 DG128, L1/L3 LCSC-s 0630-as tekercs, kis ESR-ű kvarcok
- bekötés változatlan (netlista 0 / 0), ellenorzes.py: 0 hiba

Co-Authored-By: Claude Opus 5.5 <noreply@anthropic.com>
Claude-Session: https://claude.ai/code/session_01KVtZMUPbtveTXy9VyJshyt
Parts:
- J1: footprint TerminalBlock_Degson:TerminalBlock_Degson_DG250-3.5-02P_1x02_P3.50mm_45Degree -> TerminalBlock_Phoenix:TerminalBlock_Phoenix_MKDS-1,5-2_1x02_P5.00mm_Horizontal; Megjegyzés D84: Degson DG250-3.5-02P – rugós, nyomógombos, 8 A (UL), 0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 -> D85: Degson DG128-5.0-02P – csavaros, 5,0 mm, 15 A (UL), 2,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
- L1: Megjegyzés D84: HPI0630-6R8 – árnyékolt, Isat 4,9 A, 53 mΩ -> D85: 0630-as árnyékolt, 6,8 µH, Isat ≥ 4,5 A – SLO0630H6R8M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
- L3: Megjegyzés D84: HPI0630-8R2 – árnyékolt, Isat 3,8 A, 59,5 mΩ (2 A-en ~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 -> D85: 0630-as árnyékolt, 8,2 µH, Isat ≥ 3,8 A, ≤ 60 mΩ – APS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
- Y1: Megjegyzés D84: Kyocera CX3225FB25000F0FZZH1 – ±20 ppm, CL = 10 pF (He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 -> D85: SX3B25.000F1010F30 (LCSC C2901684) – CL = 10 pF, ESR ≤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
Changed lines of the file:
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@@
 			)
 		)
-		(property "Footprint" "TerminalBlock_Degson:TerminalBlock_Degson_DG250-3.5-02P_1x02_P3.50mm_45Degree"
+		(property "Footprint" "TerminalBlock_Phoenix:TerminalBlock_Phoenix_MKDS-1,5-2_1x02_P5.00mm_Horizontal"
 			(at 27.94 55.88 0)
 			(hide yes)
@@
 			)
 		)
-		(property "Megjegyzés" "D84: Degson DG250-3.5-02P – rugós, nyomógombos, 8 A (UL), 0,2–1,5 mm²; Hestore 100.441.02"
+		(property "Megjegyzés" "D85: Degson DG128-5.0-02P – csavaros, 5,0 mm, 15 A (UL), 2,5 mm² (mint a LED-modul J201-e)"
 			(at 27.94 55.88 0)
 			(hide yes)
@@
 			)
 		)
-		(property "Megjegyzés" "D84: Kyocera CX3225FB25000F0FZZH1 – ±20 ppm, CL = 10 pF (Hestore 100.494.61)"
+		(property "Megjegyzés" "D85: SX3B25.000F1010F30 (LCSC C2901684) – CL = 10 pF, ESR ≤ 30 Ω; vagy Kyocera CX3225FB25000F0FZZH1"
 			(at 330.2 237.49 90)
 			(hide yes)
@@
 			)
 		)
-		(property "Megjegyzés" "D84: HPI0630-8R2 – árnyékolt, Isat 3,8 A, 59,5 mΩ (2 A-en ~0,24 W)"
+		(property "Megjegyzés" "D85: 0630-as árnyékolt, 8,2 µH, Isat ≥ 3,8 A, ≤ 60 mΩ – APS0630M8R2A (LCSC) vagy HPI0630-8R2 (Hestore)"
 			(at 240.03 48.26 90)
 			(hide yes)
@@
 			)
 		)
-		(property "Megjegyzés" "D84: HPI0630-6R8 – árnyékolt, Isat 4,9 A, 53 mΩ"
+		(property "Megjegyzés" "D85: 0630-as árnyékolt, 6,8 µH, Isat ≥ 4,5 A – SLO0630H6R8MTT (LCSC) vagy HPI0630-6R8 (Hestore)"
 			(at 128.27 114.3 90)
 			(hide yes)

Commit message: Hardver: kézzel átrendezett kapcsolási rajzok (D67), védelem a generátor felülírása ellen; rajzdátum 10-23
- mind az öt lap kézi szerkesztésű – gen/kezi-lapok.txt; a build.sh ezeket nem generálja újra, csak ellenőrzi (felülírás: --force)
- bekötés változatlan (netlista 0 / 0), ERC rendben, ellenorzes.py: 0 hiba
- komponenslista: állapot 10-23

Co-Authored-By: Claude Opus 5.5 <noreply@anthropic.com>
Claude-Session: https://claude.ai/code/session_01KVtZMUPbtveTXy9VyJshyt
Other:
- note removed: "Generálva (hardware/gen/vezerlo.py) – a VEZERLO-SPEC.md alapján; kézi szerkesztés helyett a generátort módosítsd."
- moved on the sheet: C19, C21, C31, C32, C33, C34, C35, C36, C37, C38, C39, C4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
