File: hardware/led-modul/led-modul.kicad_sch (KiCad schematic)
At the start: 128 parts, among them J201 24V IN 20A, J202 BLOKK 1, J203 BLOKK 2, J204 BLOKK 3, Q201 NTMFS5C604NL, Q202 NTD5C648NL, Q203 NTD5C648NL, Q204 NTD5C648NL, Q205 NTD5C648NL, Q206 NTD5C648NL, Q207 NTD5C648NL, U201 UCC27524DR, U202 UCC27524DR, U203 UCC27524DR, U205 MC78L12ACDR2G, U206 INA181A2IDBVR, U207 MCP9701AT-E/TT

Commit message: Hardver: legolcsóbb beszerzés (D84) – Hestore + DigiKey, a rajz a kapható típusokra igazítva; beszerzési lista
- gen/beszerzes.py → bom/beszerzes.csv: BOM-tételenként forrás, Hestore-kód, nettó ár, készlet
- J1/J100 Degson DG250, J201 DG128 (15 A), J202–J204 KF128, F201 15 A; L1/L3 HPI0630 (saját footprint);
  R209 CRE2512; C40/C41 12 pF; ESP32-C6-WROOM-1-N8; SS56C, BAT54HT1G, STPS3L60U, BLM18EG221
- NYÁK-ok újragenerálva (a layout még nem indult el); bekötés változatlan, ellenorzes.py: 0 hiba
- SAMPLE-KERESEK: az NTMFS5C604NL nincs kézben (javítva)

Co-Authored-By: Claude Opus 5.5 <noreply@anthropic.com>
Claude-Session: https://claude.ai/code/session_01KVtZMUPbtveTXy9VyJshyt
Parts:
- D211, D212, D213, D214, D215, D216: value B360B -> STPS3L60U
- F201: value 20A -> 15A; Megjegyzés mini lapos autós biztosíték, NYÁK-foglalat -> mini lapos autós biztosíték (normál mini, pl. Littelfuse 02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
- J201: value 24V IN 20A -> 24V IN 15A; footprint TerminalBlock_Phoenix:TerminalBlock_Phoenix_MKDS-3-2-5.08_1x02_P5.08mm_Horizontal -> TerminalBlock_Phoenix:TerminalBlock_Phoenix_MKDS-1,5-2_1x02_P5.00mm_Horizontal; Megjegyzés csavaros (Phoenix MKDS 3, 5,08 mm, 24 A / 4 mm²) – D79; bar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 -> csavaros, liftes: Degson DG128-5.0-02P (5,0 mm, 15 A UL / 1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
- J202: footprint TerminalBlock_Phoenix:TerminalBlock_Phoenix_MKDS-3-3-5.08_1x03_P5.08mm_Horizontal -> TerminalBlock_Phoenix:TerminalBlock_Phoenix_MKDS-1,5-3_1x03_P5.00mm_Horizontal; Megjegyzés 1 = +24 V, 2 = CH1, 3 = CH2; csavaros (MKDS 3, 5,08 mm) – D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 -> 1 = +24 V, 2 = CH1, 3 = CH2; csavaros, KF128-5.0-3P (5,0 mm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
- J203: footprint TerminalBlock_Phoenix:TerminalBlock_Phoenix_MKDS-3-3-5.08_1x03_P5.08mm_Horizontal -> TerminalBlock_Phoenix:TerminalBlock_Phoenix_MKDS-1,5-3_1x03_P5.00mm_Horizontal; Megjegyzés 1 = +24 V, 2 = CH3, 3 = CH4; csavaros (MKDS 3, 5,08 mm) – D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 -> 1 = +24 V, 2 = CH3, 3 = CH4; csavaros, KF128-5.0-3P (5,0 mm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
- J204: footprint TerminalBlock_Phoenix:TerminalBlock_Phoenix_MKDS-3-3-5.08_1x03_P5.08mm_Horizontal -> TerminalBlock_Phoenix:TerminalBlock_Phoenix_MKDS-1,5-3_1x03_P5.00mm_Horizontal; Megjegyzés 1 = +24 V, 2 = CH5, 3 = CH6; csavaros (MKDS 3, 5,08 mm) – D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 -> 1 = +24 V, 2 = CH5, 3 = CH6; csavaros, KF128-5.0-3P (5,0 mm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
- R209: Megjegyzés 2512, ≥ 1 W (20 A-en 0,4 W), Kelvin – pl. Vishay WSK2512 / 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 -> D84: Bourns CRE2512-FZ-R001E-3 (2512, 3 W; 15 A-en 0,23 W) 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
Other:
- note added: "1. BETÁP (15 A): J201 → F201 15 A → +24V_RAIL; fordított polaritás ellen Q201 N-FET a GND-ágban (D78) – a közös föld miatt a + ági védelem nem elég"
- note added: "3. CSATORNÁK (× 6): FET NTD5C648NL (DPAK; tartalék IRFR1205) · szabadonfutó STPS3L60U a blokk +24 V-jára · RC snubber (DNP) · gate-LED + drain-LED · drain → ADC osztó"
- note removed: "1. BETÁP (20 A): J201 → F201 20 A → +24V_RAIL; fordított polaritás ellen Q201 N-FET a GND-ágban (D78) – a közös föld miatt a + ági védelem nem elég"
- note removed: "3. CSATORNÁK (× 6): FET NTD5C648NL (DPAK; tartalék IRFR1205) · szabadonfutó B360B a blokk +24 V-jára · RC snubber (DNP) · gate-LED + drain-LED · drain → ADC osztó"
- title: LED-modul – 6 × 10 A low-side PWM (össz. 20 A), modulmag -> LED-modul – 6 × 10 A low-side PWM (össz. 15 A), modulmag
Changed lines of the file:
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@@
 	(paper "A3")
 	(title_block
-		(title "LED-modul – 6 × 10 A low-side PWM (össz. 20 A), modulmag")
+		(title "LED-modul – 6 × 10 A low-side PWM (össz. 15 A), modulmag")
 		(date "2026-10-22")
 		(rev "v1 vázlat")
@@
 		)
 	)
-	(text "1. BETÁP (20 A): J201 → F201 20 A → +24V_RAIL; fordított polaritás ellen Q201 N-FET a GND-ágban (D78) – a közös föld miatt a + ági védelem nem elég"
+	(text "1. BETÁP (15 A): J201 → F201 15 A → +24V_RAIL; fordított polaritás ellen Q201 N-FET a GND-ágban (D78) – a közös föld miatt a + ági védelem nem elég"
 		(exclude_from_sim no)
 		(at 80 24 0)
@@
 		)
 	)
-	(text "3. CSATORNÁK (× 6): FET NTD5C648NL (DPAK; tartalék IRFR1205) · szabadonfutó B360B a blokk +24 V-jára · RC snubber (DNP) · gate-LED + drain-LED · drain → ADC osztó"
+	(text "3. CSATORNÁK (× 6): FET NTD5C648NL (DPAK; tartalék IRFR1205) · szabadonfutó STPS3L60U a blokk +24 V-jára · RC snubber (DNP) · gate-LED + drain-LED · drain → ADC osztó"
 		(exclude_from_sim no)
 		(at 15 146.75 0)
@@
 			)
 		)
-		(property "Megjegyzés" "2512, ≥ 1 W (20 A-en 0,4 W), Kelvin – pl. Vishay WSK2512 / WSLP2512"
+		(property "Megjegyzés" "D84: Bourns CRE2512-FZ-R001E-3 (2512, 3 W; 15 A-en 0,23 W) – 2 kivezetésű: a Kelvin-padokon összeforrasztva"
 			(at 39.37 256.54 0)
 			(hide yes)
@@
 			)
 		)
-		(property "Footprint" "TerminalBlock_Phoenix:TerminalBlock_Phoenix_MKDS-3-3-5.08_1x03_P5.08mm_Horizontal"
+		(property "Footprint" "TerminalBlock_Phoenix:TerminalBlock_Phoenix_MKDS-1,5-3_1x03_P5.00mm_Horizontal"
 			(at 339.09 67.31 0)
 			(hide yes)
@@
 			)
 		)
-		(property "Megjegyzés" "1 = +24 V, 2 = CH3, 3 = CH4; csavaros (MKDS 3, 5,08 mm) – D79"
+		(property "Megjegyzés" "1 = +24 V, 2 = CH3, 3 = CH4; csavaros, KF128-5.0-3P (5,0 mm, 10 A – a blokkbiztosíték ≤ 10 A) – D84"
 			(at 339.09 67.31 0)
 			(hide yes)
@@
 			)
 		)
-		(property "Value" "B360B"
+		(property "Value" "STPS3L60U"
 			(at 173.99 166.37 90)
 			(show_name no)
@@
 			)
 		)
-		(property "Value" "B360B"
+		(property "Value" "STPS3L60U"
 			(at 367.03 166.37 90)
 			(show_name no)
@@
 			)
 		)
-		(property "Value" "24V IN 20A"
+		(property "Value" "24V IN 15A"
 			(at 87.63 54.61 0)
 			(show_name no)
@@
 			)
 		)
-		(property "Footprint" "TerminalBlock_Phoenix:TerminalBlock_Phoenix_MKDS-3-2-5.08_1x02_P5.08mm_Horizontal"
+		(property "Footprint" "TerminalBlock_Phoenix:TerminalBlock_Phoenix_MKDS-1,5-2_1x02_P5.00mm_Horizontal"
 			(at 90.17 59.69 0)
 			(hide yes)
@@
 			)
 		)
-		(property "Megjegyzés" "csavaros (Phoenix MKDS 3, 5,08 mm, 24 A / 4 mm²) – D79; barna = +24 V, kék = GND (D43)"
+		(property "Megjegyzés" "csavaros, liftes: Degson DG128-5.0-02P (5,0 mm, 15 A UL / 18 A IEC, 2,5 mm²) – D84; barna = +24 V, kék = GND (D43)"
 			(at 90.17 59.69 0)
 			(hide yes)
@@
 			)
 		)
-		(property "Value" "B360B"
+		(property "Value" "STPS3L60U"
 			(at 46.99 166.37 90)
 			(show_name no)
@@
 			)
 		)
-		(property "Value" "B360B"
+		(property "Value" "STPS3L60U"
 			(at 302.26 166.37 90)
 			(show_name no)
@@
 			)
 		)
-		(property "Value" "B360B"
+		(property "Value" "STPS3L60U"
 			(at 110.49 166.37 90)
 			(show_name no)
@@
 			)
 		)
-		(property "Footprint" "TerminalBlock_Phoenix:TerminalBlock_Phoenix_MKDS-3-3-5.08_1x03_P5.08mm_Horizontal"
+		(property "Footprint" "TerminalBlock_Phoenix:TerminalBlock_Phoenix_MKDS-1,5-3_1x03_P5.00mm_Horizontal"
 			(at 372.11 67.31 0)
 			(hide yes)
@@
 			)
 		)
-		(property "Megjegyzés" "1 = +24 V, 2 = CH5, 3 = CH6; csavaros (MKDS 3, 5,08 mm) – D79"
+		(property "Megjegyzés" "1 = +24 V, 2 = CH5, 3 = CH6; csavaros, KF128-5.0-3P (5,0 mm, 10 A – a blokkbiztosíték ≤ 10 A) – D84"
 			(at 372.11 67.31 0)
 			(hide yes)
@@
 			)
 		)
-		(property "Value" "B360B"
+		(property "Value" "STPS3L60U"
 			(at 238.76 166.37 90)
 			(show_name no)
@@
 			)
 		)
-		(property "Footprint" "TerminalBlock_Phoenix:TerminalBlock_Phoenix_MKDS-3-3-5.08_1x03_P5.08mm_Horizontal"
+		(property "Footprint" "TerminalBlock_Phoenix:TerminalBlock_Phoenix_MKDS-1,5-3_1x03_P5.00mm_Horizontal"
 			(at 306.07 67.31 0)
 			(hide yes)
@@
 			)
 		)
-		(property "Megjegyzés" "1 = +24 V, 2 = CH1, 3 = CH2; csavaros (MKDS 3, 5,08 mm) – D79"
+		(property "Megjegyzés" "1 = +24 V, 2 = CH1, 3 = CH2; csavaros, KF128-5.0-3P (5,0 mm, 10 A – a blokkbiztosíték ≤ 10 A) – D84"
 			(at 306.07 67.31 0)
 			(hide yes)
@@
 			)
 		)
-		(property "Value" "20A"
+		(property "Value" "15A"
 			(at 93.98 46.99 90)
 			(show_name no)
@@
 			)
 		)
-		(property "Megjegyzés" "mini lapos autós biztosíték, NYÁK-foglalat"
+		(property "Megjegyzés" "mini lapos autós biztosíték (normál mini, pl. Littelfuse 0297015), Keystone 3568 foglalat; 15 A = a J201 névleges árama (D84)"
 			(at 93.98 44.45 90)
 			(hide yes)
