File: hardware/led-modul/led-modul.kicad_sch (KiCad schematic)
At the start: 128 parts, among them J201 24V IN 15A, J202 BLOKK 1, J203 BLOKK 2, J204 BLOKK 3, Q201 NTMFS5C604NL, Q202 NTD5C648NL, Q203 NTD5C648NL, Q204 NTD5C648NL, Q205 NTD5C648NL, Q206 NTD5C648NL, Q207 NTD5C648NL, U201 UCC27524DR, U202 UCC27524DR, U203 UCC27524DR, U205 MC78L12ACDR2G, U206 INA181A2IDBVR, U207 MCP9701AT-E/TT

Commit message: Hardver: legolcsóbb beszerzés LCSC-ről (D85), megszűnt FET-ek pótlása, LCSC-kosárlista
- gen/lcsc.py: LCSC-árak a JLC alkatrészkeresőjéből; gen/beszerzes.py soronként a legolcsóbb forrás (Hestore / LCSC, ÁFA-val)
- bom/lcsc-kosar.csv: 99 tétel (~15 eFt), az LCSC BOM Tooljába feltölthető; házak később, ST-Link/Nucleo kézben
- Q202–Q207 NTD5C648NL → NCE6080K, Q201 NTMFS5C604NL → NCEP6090AGU (nem kaphatók), F201 → NANO² 15 A,
  D211–D216 SS56B, J1/J100 DG128, L1/L3 LCSC-s 0630-as tekercs, kis ESR-ű kvarcok
- bekötés változatlan (netlista 0 / 0), ellenorzes.py: 0 hiba

Co-Authored-By: Claude Opus 5.5 <noreply@anthropic.com>
Claude-Session: https://claude.ai/code/session_01KVtZMUPbtveTXy9VyJshyt
Parts:
- D211, D212, D213, D214, D215, D216: value STPS3L60U -> SS56B; Megjegyzés szabadonfutó, 3 A / 60 V, SMB -> szabadonfutó, 5 A / 60 V, SMB (D85)
- F201: footprint Fuse:Fuseholder_Blade_Mini_Keystone_3568 -> Fuse:Fuse_Littelfuse-NANO2-451_453; Megjegyzés mini lapos autós biztosíték (normál mini, pl. Littelfuse 02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 -> D85: Littelfuse 0451015.MRL (NANO² 15 A, 2410) – beforraszt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
- Q201: value NTMFS5C604NL -> NCEP6090AGU; Megjegyzés onsemi 60 V, ~1,2 mΩ, SO-8FL; D = GND_IN (J201), S = GND; n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 -> D85: NCE 60 V, 2,8 mΩ, DFN5×6 (power-SO8, az SO-8FL padképé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
- Q202, Q203, Q204, Q205, Q206, Q207: value NTD5C648NL -> NCE6080K; Megjegyzés onsemi 60 V, ~4–5 mΩ, DPAK; tartalék: IRFR1205 (kis áramra) -> D85: NCE 60 V, 8,5 mΩ @ 10 V, DPAK (az NTD5C648NL megszűnt)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
Other:
- note added: "3. CSATORNÁK (× 6): FET NCE6080K (DPAK; tartalék IRFR1205) · szabadonfutó SS56B a blokk +24 V-jára · RC snubber (DNP) · gate-LED + drain-LED · drain → ADC osztó"
- note removed: "3. CSATORNÁK (× 6): FET NTD5C648NL (DPAK; tartalék IRFR1205) · szabadonfutó STPS3L60U a blokk +24 V-jára · RC snubber (DNP) · gate-LED + drain-LED · drain → ADC osztó"
Changed lines of the file:
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@@
 		)
 	)
-	(text "3. CSATORNÁK (× 6): FET NTD5C648NL (DPAK; tartalék IRFR1205) · szabadonfutó STPS3L60U a blokk +24 V-jára · RC snubber (DNP) · gate-LED + drain-LED · drain → ADC osztó"
+	(text "3. CSATORNÁK (× 6): FET NCE6080K (DPAK; tartalék IRFR1205) · szabadonfutó SS56B a blokk +24 V-jára · RC snubber (DNP) · gate-LED + drain-LED · drain → ADC osztó"
 		(exclude_from_sim no)
 		(at 15 146.75 0)
@@
 			)
 		)
-		(property "Value" "NTD5C648NL"
+		(property "Value" "NCE6080K"
 			(at 302.26 196.85 0)
 			(show_name no)
@@
 			)
 		)
-		(property "Description" "N-MOSFET 60 V, DPAK (onsemi NTD5C648NL)"
+		(property "Description" "N-MOSFET 60 V, DPAK (NCE NCE6080K)"
 			(at 297.18 190.5 0)
 			(hide yes)
@@
 			)
 		)
-		(property "Megjegyzés" "onsemi 60 V, ~4–5 mΩ, DPAK; tartalék: IRFR1205 (kis áramra)"
+		(property "Megjegyzés" "D85: NCE 60 V, 8,5 mΩ @ 10 V, DPAK (az NTD5C648NL megszűnt); 10 A-en ~0,85 W; tartalék: IRFR1205"
 			(at 297.18 190.5 0)
 			(hide yes)
@@
 			)
 		)
-		(property "Value" "NTMFS5C604NL"
+		(property "Value" "NCEP6090AGU"
 			(at 125.73 67.31 0)
 			(show_name no)
@@
 			)
 		)
-		(property "Description" "N-MOSFET 60 V, ~1,2 mΩ (onsemi NTMFS5C604NL)"
+		(property "Description" "N-MOSFET 60 V, 2,8 mΩ (NCE NCEP6090AGU)"
 			(at 119.38 66.04 0)
 			(hide yes)
@@
 			)
 		)
-		(property "Megjegyzés" "onsemi 60 V, ~1,2 mΩ, SO-8FL; D = GND_IN (J201), S = GND; nagy padek (áthidalható)"
+		(property "Megjegyzés" "D85: NCE 60 V, 2,8 mΩ, DFN5×6 (power-SO8, az SO-8FL padképére; az NTMFS5C604NL nem kapható); D = GND_IN (J201), S = GND"
 			(at 119.38 66.04 0)
 			(hide yes)
@@
 			)
 		)
-		(property "Value" "NTD5C648NL"
+		(property "Value" "NCE6080K"
 			(at 110.49 196.85 0)
 			(show_name no)
@@
 			)
 		)
-		(property "Description" "N-MOSFET 60 V, DPAK (onsemi NTD5C648NL)"
+		(property "Description" "N-MOSFET 60 V, DPAK (NCE NCE6080K)"
 			(at 105.41 190.5 0)
 			(hide yes)
@@
 			)
 		)
-		(property "Megjegyzés" "onsemi 60 V, ~4–5 mΩ, DPAK; tartalék: IRFR1205 (kis áramra)"
+		(property "Megjegyzés" "D85: NCE 60 V, 8,5 mΩ @ 10 V, DPAK (az NTD5C648NL megszűnt); 10 A-en ~0,85 W; tartalék: IRFR1205"
 			(at 105.41 190.5 0)
 			(hide yes)
@@
 			)
 		)
-		(property "Value" "NTD5C648NL"
+		(property "Value" "NCE6080K"
 			(at 46.99 196.85 0)
 			(show_name no)
@@
 			)
 		)
-		(property "Description" "N-MOSFET 60 V, DPAK (onsemi NTD5C648NL)"
+		(property "Description" "N-MOSFET 60 V, DPAK (NCE NCE6080K)"
 			(at 41.91 190.5 0)
 			(hide yes)
@@
 			)
 		)
-		(property "Megjegyzés" "onsemi 60 V, ~4–5 mΩ, DPAK; tartalék: IRFR1205 (kis áramra)"
+		(property "Megjegyzés" "D85: NCE 60 V, 8,5 mΩ @ 10 V, DPAK (az NTD5C648NL megszűnt); 10 A-en ~0,85 W; tartalék: IRFR1205"
 			(at 41.91 190.5 0)
 			(hide yes)
@@
 			)
 		)
-		(property "Value" "STPS3L60U"
+		(property "Value" "SS56B"
 			(at 173.99 166.37 90)
 			(show_name no)
@@
 			)
 		)
-		(property "Megjegyzés" "szabadonfutó, 3 A / 60 V, SMB"
+		(property "Megjegyzés" "szabadonfutó, 5 A / 60 V, SMB (D85)"
 			(at 171.45 165.1 90)
 			(hide yes)
@@
 			)
 		)
-		(property "Value" "NTD5C648NL"
+		(property "Value" "NCE6080K"
 			(at 173.99 196.85 0)
 			(show_name no)
@@
 			)
 		)
-		(property "Description" "N-MOSFET 60 V, DPAK (onsemi NTD5C648NL)"
+		(property "Description" "N-MOSFET 60 V, DPAK (NCE NCE6080K)"
 			(at 168.91 190.5 0)
 			(hide yes)
@@
 			)
 		)
-		(property "Megjegyzés" "onsemi 60 V, ~4–5 mΩ, DPAK; tartalék: IRFR1205 (kis áramra)"
+		(property "Megjegyzés" "D85: NCE 60 V, 8,5 mΩ @ 10 V, DPAK (az NTD5C648NL megszűnt); 10 A-en ~0,85 W; tartalék: IRFR1205"
 			(at 168.91 190.5 0)
 			(hide yes)
@@
 			)
 		)
-		(property "Value" "STPS3L60U"
+		(property "Value" "SS56B"
 			(at 367.03 166.37 90)
 			(show_name no)
@@
 			)
 		)
-		(property "Megjegyzés" "szabadonfutó, 3 A / 60 V, SMB"
+		(property "Megjegyzés" "szabadonfutó, 5 A / 60 V, SMB (D85)"
 			(at 364.49 165.1 90)
 			(hide yes)
@@
 			)
 		)
-		(property "Value" "STPS3L60U"
+		(property "Value" "SS56B"
 			(at 46.99 166.37 90)
 			(show_name no)
@@
 			)
 		)
-		(property "Megjegyzés" "szabadonfutó, 3 A / 60 V, SMB"
+		(property "Megjegyzés" "szabadonfutó, 5 A / 60 V, SMB (D85)"
 			(at 44.45 165.1 90)
 			(hide yes)
@@
 			)
 		)
-		(property "Value" "STPS3L60U"
+		(property "Value" "SS56B"
 			(at 302.26 166.37 90)
 			(show_name no)
@@
 			)
 		)
-		(property "Megjegyzés" "szabadonfutó, 3 A / 60 V, SMB"
+		(property "Megjegyzés" "szabadonfutó, 5 A / 60 V, SMB (D85)"
 			(at 299.72 165.1 90)
 			(hide yes)
@@
 			)
 		)
-		(property "Value" "NTD5C648NL"
+		(property "Value" "NCE6080K"
 			(at 367.03 196.85 0)
 			(show_name no)
@@
 			)
 		)
-		(property "Description" "N-MOSFET 60 V, DPAK (onsemi NTD5C648NL)"
+		(property "Description" "N-MOSFET 60 V, DPAK (NCE NCE6080K)"
 			(at 361.95 190.5 0)
 			(hide yes)
@@
 			)
 		)
-		(property "Megjegyzés" "onsemi 60 V, ~4–5 mΩ, DPAK; tartalék: IRFR1205 (kis áramra)"
+		(property "Megjegyzés" "D85: NCE 60 V, 8,5 mΩ @ 10 V, DPAK (az NTD5C648NL megszűnt); 10 A-en ~0,85 W; tartalék: IRFR1205"
 			(at 361.95 190.5 0)
 			(hide yes)
@@
 			)
 		)
-		(property "Value" "STPS3L60U"
+		(property "Value" "SS56B"
 			(at 110.49 166.37 90)
 			(show_name no)
@@
 			)
 		)
-		(property "Megjegyzés" "szabadonfutó, 3 A / 60 V, SMB"
+		(property "Megjegyzés" "szabadonfutó, 5 A / 60 V, SMB (D85)"
 			(at 107.95 165.1 90)
 			(hide yes)
@@
 			)
 		)
-		(property "Value" "NTD5C648NL"
+		(property "Value" "NCE6080K"
 			(at 238.76 196.85 0)
 			(show_name no)
@@
 			)
 		)
-		(property "Description" "N-MOSFET 60 V, DPAK (onsemi NTD5C648NL)"
+		(property "Description" "N-MOSFET 60 V, DPAK (NCE NCE6080K)"
 			(at 233.68 190.5 0)
 			(hide yes)
@@
 			)
 		)
-		(property "Megjegyzés" "onsemi 60 V, ~4–5 mΩ, DPAK; tartalék: IRFR1205 (kis áramra)"
+		(property "Megjegyzés" "D85: NCE 60 V, 8,5 mΩ @ 10 V, DPAK (az NTD5C648NL megszűnt); 10 A-en ~0,85 W; tartalék: IRFR1205"
 			(at 233.68 190.5 0)
 			(hide yes)
@@
 			)
 		)
-		(property "Value" "STPS3L60U"
+		(property "Value" "SS56B"
 			(at 238.76 166.37 90)
 			(show_name no)
@@
 			)
 		)
-		(property "Megjegyzés" "szabadonfutó, 3 A / 60 V, SMB"
+		(property "Megjegyzés" "szabadonfutó, 5 A / 60 V, SMB (D85)"
 			(at 236.22 165.1 90)
 			(hide yes)
@@
 			)
 		)
-		(property "Footprint" "Fuse:Fuseholder_Blade_Mini_Keystone_3568"
+		(property "Footprint" "Fuse:Fuse_Littelfuse-NANO2-451_453"
 			(at 93.98 44.45 90)
 			(hide yes)
@@
 			)
 		)
-		(property "Megjegyzés" "mini lapos autós biztosíték (normál mini, pl. Littelfuse 0297015), Keystone 3568 foglalat; 15 A = a J201 névleges árama (D84)"
+		(property "Megjegyzés" "D85: Littelfuse 0451015.MRL (NANO² 15 A, 2410) – beforrasztott; 15 A = a J201 névleges árama (D84)"
 			(at 93.98 44.45 90)
 			(hide yes)

Commit message: Hardver: kézzel átrendezett kapcsolási rajzok (D67), védelem a generátor felülírása ellen; rajzdátum 10-23
- mind az öt lap kézi szerkesztésű – gen/kezi-lapok.txt; a build.sh ezeket nem generálja újra, csak ellenőrzi (felülírás: --force)
- bekötés változatlan (netlista 0 / 0), ERC rendben, ellenorzes.py: 0 hiba
- komponenslista: állapot 10-23

Co-Authored-By: Claude Opus 5.5 <noreply@anthropic.com>
Claude-Session: https://claude.ai/code/session_01KVtZMUPbtveTXy9VyJshyt
Other:
- note removed: "Generálva (hardware/gen/led-modul.py) – D43/D47/D53/D65 alapján; kézi szerkesztés helyett a generátort módosítsd."
Changed lines of the file:
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@@
 	(title_block
 		(title "LED-modul – 6 × 10 A low-side PWM (össz. 15 A), modulmag")
-		(date "2026-10-22")
+		(date "2026-10-23")
 		(rev "v1 vázlat")
 		(company "Moduláris okosotthon platform – szakdolgozat")
@@
 		)
 	)
-	(text "Generálva (hardware/gen/led-modul.py) – D43/D47/D53/D65 alapján; kézi szerkesztés helyett a generátort módosítsd."
-		(exclude_from_sim no)
-		(at 15 281 0)
-		(effects
-			(font
-				(size 1.3 1.3)
-			)
-			(justify left bottom)
-		)
-	)
 	(text "a 24 V-ot a PB1 méri, a főbiztosíték előtt"
 		(exclude_from_sim no)
@@
 	)
 	(junction
-		(at 125.73 44.45)
-		(diameter 0)
-		(color 0 0 0 0)
-	)
-	(junction
 		(at 199.39 248.92)
 		(diameter 0)
@@
 	(wire
 		(pts
-			(xy 125.73 44.45) (xy 130.81 44.45)
-		)
-		(stroke
-			(width 0)
-			(type default)
-		)
-	)
-	(wire
-		(pts
 			(xy 242.57 44.45) (xy 242.57 54.61)
 		)
@@
 	(wire
 		(pts
-			(xy 97.79 44.45) (xy 125.73 44.45)
+			(xy 97.79 44.45) (xy 130.81 44.45)
 		)
 		(stroke
@@
 		)
 	)
+	(embedded_fonts no)
 )
