File: hardware/bemeneti-modul/bemeneti-modul.kicad_sch (KiCad schematic)
At the start: 113 parts, among them J301 IN0, J302 IN1, J303 IN2, J304 IN3, J305 IN4, J306 IN5, J307 IN6, J308 IN7, J309 IN8, J310 IN9, J311 IN10, J312 IN11, J313 IN12, J314 IN13, J315 IN14, J316 IN15, J320 I2C KÜLSŐ, U301 AP2112K-3.3TRG1, U302 HDC3020DEFR, U303 TPD4E05U06DQAR, U304 TPD4E05U06DQAR, U305 TPD4E05U06DQAR, U306 TPD4E05U06DQAR, U307 TPD4E05U06DQAR

Commit message: Hardver: kézzel átrendezett kapcsolási rajzok (D67), védelem a generátor felülírása ellen; rajzdátum 10-23
- mind az öt lap kézi szerkesztésű – gen/kezi-lapok.txt; a build.sh ezeket nem generálja újra, csak ellenőrzi (felülírás: --force)
- bekötés változatlan (netlista 0 / 0), ERC rendben, ellenorzes.py: 0 hiba
- komponenslista: állapot 10-23

Co-Authored-By: Claude Opus 5.5 <noreply@anthropic.com>
Claude-Session: https://claude.ai/code/session_01KVtZMUPbtveTXy9VyJshyt
Other:
- note removed: "Generálva (hardware/gen/bemeneti-modul.py) – D44/D48/D51/D66 alapján; kézi szerkesztés helyett a generátort módosítsd."
- moved on the sheet: C301, R301, R302, R390
Changed lines of the file:
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@@
 	(title_block
 		(title "Bemeneti modul – 16 bemenet, 4 tápcsoport, HDC3020")
-		(date "2026-10-22")
+		(date "2026-10-23")
 		(rev "v1 vázlat")
 		(company "Moduláris okosotthon platform – szakdolgozat")
@@
 	(text "HW-ID: bemeneti modul = 3. sáv (0,66 V)"
 		(exclude_from_sim no)
-		(at 12 112 0)
+		(at 18.35 112 0)
 		(effects
 			(font
@@
 		)
 	)
-	(text "Generálva (hardware/gen/bemeneti-modul.py) – D44/D48/D51/D66 alapján; kézi szerkesztés helyett a generátort módosítsd."
-		(exclude_from_sim no)
-		(at 15 281 0)
-		(effects
-			(font
-				(size 1.3 1.3)
-			)
-			(justify left bottom)
-		)
-	)
 	(text "IN4–IN7"
 		(exclude_from_sim no)
@@
 	)
 	(junction
-		(at 38.1 128.27)
+		(at 44.45 128.27)
 		(diameter 0)
 		(color 0 0 0 0)
@@
 	)
 	(junction
-		(at 20.32 128.27)
+		(at 26.67 128.27)
 		(diameter 0)
 		(color 0 0 0 0)
@@
 	(wire
 		(pts
-			(xy 20.32 128.27) (xy 38.1 128.27)
+			(xy 26.67 128.27) (xy 44.45 128.27)
 		)
 		(stroke
@@
 	(wire
 		(pts
-			(xy 38.1 128.27) (xy 38.1 130.81)
+			(xy 44.45 128.27) (xy 44.45 130.81)
 		)
 		(stroke
@@
 	(wire
 		(pts
-			(xy 20.32 149.86) (xy 22.86 149.86)
+			(xy 26.67 149.86) (xy 29.21 149.86)
 		)
 		(stroke
@@
 	(wire
 		(pts
-			(xy 20.32 125.73) (xy 20.32 128.27)
+			(xy 26.67 125.73) (xy 26.67 128.27)
 		)
 		(stroke
@@
 	(wire
 		(pts
-			(xy 20.32 128.27) (xy 20.32 130.81)
+			(xy 26.67 128.27) (xy 26.67 130.81)
 		)
 		(stroke
@@
 	(wire
 		(pts
-			(xy 30.48 149.86) (xy 33.02 149.86)
+			(xy 36.83 149.86) (xy 39.37 149.86)
 		)
 		(stroke
@@
 	(wire
 		(pts
-			(xy 38.1 128.27) (xy 43.18 128.27)
+			(xy 44.45 128.27) (xy 49.53 128.27)
 		)
 		(stroke
@@
 	(wire
 		(pts
-			(xy 33.02 149.86) (xy 33.02 152.4)
+			(xy 39.37 149.86) (xy 39.37 152.4)
 		)
 		(stroke
@@
 	)
 	(label "GND_BUS"
-		(at 20.32 149.86 180)
+		(at 26.67 149.86 180)
 		(effects
 			(font
@@
 	)
 	(label "HW_ID"
-		(at 43.18 128.27 0)
+		(at 49.53 128.27 0)
 		(effects
 			(font
@@
 	(symbol
 		(lib_id "Device:R")
-		(at 26.67 149.86 90)
+		(at 33.02 149.86 90)
 		(unit 1)
 		(body_style 1)
@@
 		(dnp no)
 		(property "Reference" "R390"
-			(at 26.67 147.32 90)
+			(at 33.02 147.32 90)
 			(show_name no)
 			(do_not_autoplace no)
@@
 		)
 		(property "Value" "0R"
-			(at 26.67 152.4 90)
+			(at 33.02 152.4 90)
 			(show_name no)
 			(do_not_autoplace no)
@@
 		)
 		(property "Footprint" "Resistor_SMD:R_1206_3216Metric"
-			(at 26.67 149.86 90)
+			(at 33.02 149.86 90)
 			(hide yes)
 			(show_name no)
@@
 		)
 		(property "Datasheet" ""
-			(at 26.67 149.86 90)
+			(at 33.02 149.86 90)
 			(hide yes)
 			(show_name no)
@@
 		)
 		(property "Description" ""
-			(at 26.67 149.86 0)
+			(at 33.02 149.86 0)
 			(show_name no)
 			(do_not_autoplace no)
@@
 		)
 		(property "Megjegyzés" "D74: 0 Ω – a bemeneti modul teljesen a buszról jár, itt ellenállás nem lehet"
-			(at 26.67 149.86 90)
+			(at 33.02 149.86 90)
 			(hide yes)
 			(show_name no)
@@
 	(symbol
 		(lib_id "power:GND")
-		(at 38.1 138.43 0)
+		(at 44.45 138.43 0)
 		(unit 1)
 		(body_style 1)
@@
 		(dnp no)
 		(property "Reference" "#PWR003"
-			(at 38.1 135.89 0)
+			(at 44.45 135.89 0)
 			(hide yes)
 			(show_name no)
@@
 		)
 		(property "Value" "GND"
-			(at 38.1 140.97 0)
+			(at 44.45 140.97 0)
 			(show_name no)
 			(do_not_autoplace no)
@@
 		)
 		(property "Footprint" ""
-			(at 38.1 138.43 0)
+			(at 44.45 138.43 0)
 			(hide yes)
 			(show_name no)
@@
 		)
 		(property "Datasheet" ""
-			(at 38.1 138.43 0)
+			(at 44.45 138.43 0)
 			(hide yes)
 			(show_name no)
@@
 		)
 		(property "Description" ""
-			(at 38.1 138.43 0)
+			(at 44.45 138.43 0)
 			(show_name no)
 			(do_not_autoplace no)
@@
 	(symbol
 		(lib_id "Device:R")
-		(at 20.32 134.62 0)
+		(at 26.67 134.62 0)
 		(unit 1)
 		(body_style 1)
@@
 		(dnp no)
 		(property "Reference" "R302"
-			(at 22.86 133.35 0)
+			(at 29.21 133.35 0)
 			(show_name no)
 			(do_not_autoplace no)
@@
 		)
 		(property "Value" "2k49 1%"
-			(at 22.86 135.89 0)
+			(at 29.21 135.89 0)
 			(show_name no)
 			(do_not_autoplace no)
@@
 		)
 		(property "Footprint" "Resistor_SMD:R_0603_1608Metric"
-			(at 20.32 134.62 0)
+			(at 26.67 134.62 0)
 			(hide yes)
 			(show_name no)
@@
 		)
 		(property "Datasheet" ""
-			(at 20.32 134.62 0)
+			(at 26.67 134.62 0)
 			(hide yes)
 			(show_name no)
@@
 		)
 		(property "Description" ""
-			(at 20.32 134.62 0)
+			(at 26.67 134.62 0)
 			(show_name no)
 			(do_not_autoplace no)
@@
 	(symbol
 		(lib_id "power:GND")
-		(at 33.02 152.4 0)
+		(at 39.37 152.4 0)
 		(unit 1)
 		(body_style 1)
@@
 		(dnp no)
 		(property "Reference" "#PWR004"
-			(at 33.02 149.86 0)
+			(at 39.37 149.86 0)
 			(hide yes)
 			(show_name no)
@@
 		)
 		(property "Value" "GND"
-			(at 33.02 154.94 0)
+			(at 39.37 154.94 0)
 			(show_name no)
 			(do_not_autoplace no)
@@
 		)
 		(property "Footprint" ""
-			(at 33.02 152.4 0)
+			(at 39.37 152.4 0)
 			(hide yes)
 			(show_name no)
@@
 		)
 		(property "Datasheet" ""
-			(at 33.02 152.4 0)
+			(at 39.37 152.4 0)
 			(hide yes)
 			(show_name no)
@@
 		)
 		(property "Description" ""
-			(at 33.02 152.4 0)
+			(at 39.37 152.4 0)
 			(show_name no)
 			(do_not_autoplace no)
@@
 	(symbol
 		(lib_id "power:GND")
-		(at 20.32 138.43 0)
+		(at 26.67 138.43 0)
 		(unit 1)
 		(body_style 1)
@@
 		(dnp no)
 		(property "Reference" "#PWR002"
-			(at 20.32 135.89 0)
+			(at 26.67 135.89 0)
 			(hide yes)
 			(show_name no)
@@
 		)
 		(property "Value" "GND"
-			(at 20.32 140.97 0)
+			(at 26.67 140.97 0)
 			(show_name no)
 			(do_not_autoplace no)
@@
 		)
 		(property "Footprint" ""
-			(at 20.32 138.43 0)
+			(at 26.67 138.43 0)
 			(hide yes)
 			(show_name no)
@@
 		)
 		(property "Datasheet" ""
-			(at 20.32 138.43 0)
+			(at 26.67 138.43 0)
 			(hide yes)
 			(show_name no)
@@
 		)
 		(property "Description" ""
-			(at 20.32 138.43 0)
+			(at 26.67 138.43 0)
 			(show_name no)
 			(do_not_autoplace no)
@@
 	(symbol
 		(lib_id "Device:C")
-		(at 38.1 134.62 0)
+		(at 44.45 134.62 0)
 		(unit 1)
 		(body_style 1)
@@
 		(dnp no)
 		(property "Reference" "C301"
-			(at 40.64 133.35 0)
+			(at 46.99 133.35 0)
 			(show_name no)
 			(do_not_autoplace no)
@@
 		)
 		(property "Value" "100n"
-			(at 40.64 135.89 0)
+			(at 46.99 135.89 0)
 			(show_name no)
 			(do_not_autoplace no)
@@
 		)
 		(property "Footprint" "Capacitor_SMD:C_0603_1608Metric"
-			(at 38.1 134.62 0)
+			(at 44.45 134.62 0)
 			(hide yes)
 			(show_name no)
@@
 		)
 		(property "Datasheet" ""
-			(at 38.1 134.62 0)
+			(at 44.45 134.62 0)
 			(hide yes)
 			(show_name no)
@@
 		)
 		(property "Description" ""
-			(at 38.1 134.62 0)
+			(at 44.45 134.62 0)
 			(show_name no)
 			(do_not_autoplace no)
@@
 	(symbol
 		(lib_id "Device:R")
-		(at 20.32 121.92 0)
+		(at 26.67 121.92 0)
 		(unit 1)
 		(body_style 1)
@@
 		(dnp no)
 		(property "Reference" "R301"
-			(at 22.86 120.65 0)
+			(at 29.21 120.65 0)
 			(show_name no)
 			(do_not_autoplace no)
@@
 		)
 		(property "Value" "10k 1%"
-			(at 22.86 123.19 0)
+			(at 29.21 123.19 0)
 			(show_name no)
 			(do_not_autoplace no)
@@
 		)
 		(property "Footprint" "Resistor_SMD:R_0603_1608Metric"
-			(at 20.32 121.92 0)
+			(at 26.67 121.92 0)
 			(hide yes)
 			(show_name no)
@@
 		)
 		(property "Datasheet" ""
-			(at 20.32 121.92 0)
+			(at 26.67 121.92 0)
 			(hide yes)
 			(show_name no)
@@
 		)
 		(property "Description" ""
-			(at 20.32 121.92 0)
+			(at 26.67 121.92 0)
 			(show_name no)
 			(do_not_autoplace no)
@@
 	(symbol
 		(lib_id "power:+3V3")
-		(at 20.32 118.11 0)
+		(at 26.67 118.11 0)
 		(unit 1)
 		(body_style 1)
@@
 		(dnp no)
 		(property "Reference" "#PWR001"
-			(at 20.32 115.57 0)
+			(at 26.67 115.57 0)
 			(hide yes)
 			(show_name no)
@@
 		)
 		(property "Value" "+3V3"
-			(at 20.32 115.57 0)
+			(at 26.67 115.57 0)
 			(show_name no)
 			(do_not_autoplace no)
@@
 		)
 		(property "Footprint" ""
-			(at 20.32 118.11 0)
+			(at 26.67 118.11 0)
 			(hide yes)
 			(show_name no)
@@
 		)
 		(property "Datasheet" ""
-			(at 20.32 118.11 0)
+			(at 26.67 118.11 0)
 			(hide yes)
 			(show_name no)
@@
 		)
 		(property "Description" ""
-			(at 20.32 118.11 0)
+			(at 26.67 118.11 0)
 			(show_name no)
 			(do_not_autoplace no)
@@
 		)
 	)
+	(embedded_fonts no)
 )
